Commit message: adjusted laser scanner positions in urdf

File: youbot_description/urdf/youbot_base/base.urdf.xacro (robot description, xacro)
@@ -104,9 +104,9 @@
 		<!-- base laser front -->
     		<xacro:hokuyo_urg04_laser name="${name}_laser_front" parent="${name}" ros_topic="scan_front" update_rate="10" min_angle="-1.57" max_angle="1.57" >
-     			 <origin xyz="0.3 0 -0.03" rpy="0 0 0" />
+     			 <origin xyz="0.33 0 -0.03" rpy="0 0 0" />
     		</xacro:hokuyo_urg04_laser>
 		<!-- base laser back -->
     		<xacro:hokuyo_urg04_laser  name="${name}_laser_back" parent="${name}" ros_topic="scan_back" update_rate="10" min_angle="1.57" max_angle="-1.57" >
-     			 <origin xyz="-0.3 0 -0.03" rpy="0 0 ${M_PI}" />
+     			 <origin xyz="-0.33 0 -0.03" rpy="0 0 ${M_PI}" />
     		</xacro:hokuyo_urg04_laser>
 	<!-- front left wheel -->

Commit message: youbot_description: adjusted scanner positions again after more precise measurement

File: youbot_description/urdf/youbot_base/base.urdf.xacro (robot description, xacro)
@@ -104,9 +104,9 @@
 		<!-- base laser front -->
     		<xacro:hokuyo_urg04_laser name="${name}_laser_front" parent="${name}" ros_topic="scan_front" update_rate="10" min_angle="-1.57" max_angle="1.57" >
-     			 <origin xyz="0.33 0 -0.03" rpy="0 0 0" />
+     			 <origin xyz="0.309 0 -0.03" rpy="0 0 0" />
     		</xacro:hokuyo_urg04_laser>
 		<!-- base laser back -->
     		<xacro:hokuyo_urg04_laser  name="${name}_laser_back" parent="${name}" ros_topic="scan_back" update_rate="10" min_angle="1.57" max_angle="-1.57" >
-     			 <origin xyz="-0.33 0 -0.03" rpy="0 0 ${M_PI}" />
+     			 <origin xyz="-0.309 0 -0.03" rpy="0 0 ${M_PI}" />
     		</xacro:hokuyo_urg04_laser>
 	<!-- front left wheel -->
