Commit message: youbot_description: fixed bug in gripper stl files

File: youbot_description/urdf/youbot_gripper/gripper.urdf.xacro (robot description, xacro)
@@ -23,5 +23,5 @@
 				<origin xyz="0 0 -0.0139" rpy="0 ${-M_PI/2} ${M_PI/2}"/>
 				<geometry>
-					<mesh filename="package://youbot_description/meshes/youbot_gripper/palm.STL" />
+					<mesh filename="package://youbot_description/meshes/youbot_gripper/palm.dae" />
 				</geometry>
 				<material name="Black" />
