Commit message: cleaned up youbot description, added meccanum wheels no urdf, added gazebo packages

File: youbot_description/robots/youbot.urdf.xacro (robot description, xacro)
@@ -1,8 +1,4 @@
 <?xml version="1.0"?>
-<robot xmlns:sensor="http://playerstage.sourceforge.net/gazebo/xmlschema/#sensor"
-       xmlns:controller="http://playerstage.sourceforge.net/gazebo/xmlschema/#controller"
-       xmlns:interface="http://playerstage.sourceforge.net/gazebo/xmlschema/#interface"
-       xmlns:xacro="http://playerstage.sourceforge.net/gazebo/xmlschema/#interface"
-       name="youbot_urdf" >
+<robot name="youbot" xmlns:xacro="http://www.ros.org/wiki/xacro">
   <!-- The following included files set up definitions of parts of the robot body -->
   <!-- misc common stuff? -->
@@ -16,52 +12,14 @@
   <!-- youbot gripper -->
   <xacro:include filename="$(find youbot_description)/urdf/youbot_gripper/gripper.urdf.xacro" />
-  <!-- generic simulator_gazebo plugins for starting mechanism control, ros time, ros battery -->
-  <xacro:include filename="$(find youbot_description)/gazebo/gazebo.urdf.xacro" />
-  <!-- materials for visualization -->
-  <xacro:include filename="$(find youbot_description)/urdf/materials.urdf.xacro" />
   <!-- Now we can start using the macros included above to define the actual youbot -->
-  <!-- The first use of a macro.  This one was defined in base.urdf.xacro above.
-       A macro like this will expand to a set of link and joint definitions, and to additional
-       Gazebo-related extensions (sensor plugins, etc).  The macro takes an argument, name,
-       that equals "base", and uses it to generate names for its component links and joints
-       (e.g., base_link).  The included origin block is also an argument to the macro.  By convention,
-       the origin block defines where the component is w.r.t its parent (in this case the parent
-       is the world frame). For more, see http://www.ros.org/wiki/xacro -->
-<!-- foot for arm-->
   <xacro:youbot_base name="base"/>
   <xacro:youbot_plate name="plate" parent="base_link">
-    <origin xyz="-0.159 0 0.046" rpy="0 0 0" />
+    <origin xyz="-0.039 0 0.064" rpy="0 0 0" />
   </xacro:youbot_plate>
   <xacro:youbot_arm name="arm" parent="base_link">
-    <origin xyz="0.143 0 0.046" rpy="0 0 0" />
+    <origin xyz="0.258 0 0.066" rpy="0 0 0.576" />
   </xacro:youbot_arm>
   <xacro:youbot_gripper name="gripper" parent="arm_link_5">
     <origin xyz="0 0 0" rpy="0 0 0" />
   </xacro:youbot_gripper>
-  <!-- BRSU SPECIFIC STUFF -->
-  <xacro:include filename="$(find youbot_description)/urdf/updated_materials.urdf.xacro" />
-  <xacro:include filename="$(find youbot_description)/urdf/misc/sensor_angle.urdf.xacro" />
-  <xacro:include filename="$(find youbot_description)/urdf/misc/cam3d_tower.urdf.xacro" />
-  <xacro:include filename="$(find youbot_description)/urdf/sensors/kinect_camera.urdf.xacro" />
-  <xacro:include filename="$(find youbot_description)/urdf/sensors/microsoft_lifecam.urdf.xacro" />
-  <xacro:include filename="$(find youbot_description)/urdf/sensors/asus_xtion_camera.urdf.xacro" />
-  <!-- Sensor angle on arm -->
-  <xacro:sensor_angle name="arm_sensor_angle" parent="arm_link_5">
-    <origin xyz="-0.002 0.0 -0.023" rpy="0.0 0.0 0.0" />
-  </xacro:sensor_angle>
-  <!-- ASUS Xtion on arm sensor angle -->
-<!--
-  <xacro:asus_xtion_camera name="openni" parent="arm_sensor_angle_part2_link"  tilt="0.0">
-    <origin xyz="0.01 0.0 0.0" rpy="${M_PI} 0.0 ${M_PI}" />
-  </xacro:asus_xtion_camera>
--->
-<!--
-  <xacro:kinect_camera name="kinect" parent="arm_link_5">
-    <origin xyz="-0.1 0.0 0.0" rpy="${M_PI} 0.0 ${M_PI}" />
-	</xacro:kinect_camera>
--->
-  <!-- Microsoft LifeCam on gripper -->
-  <xacro:microsoft_lifecam name="microsoft_lifecam" parent="arm_sensor_angle_part2_link">
-    <origin xyz="-0.04 0 -0.03" rpy="0 ${M_PI} 0" />
-  </xacro:microsoft_lifecam>
 </robot>

File: youbot_description/robots/youbot_base.urdf.xacro (robot description, xacro)
@@ -1,8 +1,4 @@
 <?xml version="1.0"?>
-<robot xmlns:sensor="http://playerstage.sourceforge.net/gazebo/xmlschema/#sensor"
-       xmlns:controller="http://playerstage.sourceforge.net/gazebo/xmlschema/#controller"
-       xmlns:interface="http://playerstage.sourceforge.net/gazebo/xmlschema/#interface"
-       xmlns:xacro="http://playerstage.sourceforge.net/gazebo/xmlschema/#interface"
-       name="youbot" >
+<robot name="youbot" xmlns:xacro="http://www.ros.org/wiki/xacro">
   <!-- The following included files set up definitions of parts of the robot body -->
   <!-- misc common stuff? -->
@@ -10,16 +6,5 @@
   <!-- youbot base -->
   <xacro:include filename="$(find youbot_description)/urdf/youbot_base/base.urdf.xacro" />
-  <!-- generic simulator_gazebo plugins for starting mechanism control, ros time, ros battery -->
-  <xacro:include filename="$(find youbot_description)/gazebo/gazebo.urdf.xacro" />
-  <!-- materials for visualization -->
-  <xacro:include filename="$(find youbot_description)/urdf/materials.urdf.xacro" />
   <!-- Now we can start using the macros included above to define the actual youbot -->
-  <!-- The first use of a macro.  This one was defined in base.urdf.xacro above.
-       A macro like this will expand to a set of link and joint definitions, and to additional
-       Gazebo-related extensions (sensor plugins, etc).  The macro takes an argument, name,
-       that equals "base", and uses it to generate names for its component links and joints
-       (e.g., base_link).  The included origin block is also an argument to the macro.  By convention,
-       the origin block defines where the component is w.r.t its parent (in this case the parent
-       is the world frame). For more, see http://www.ros.org/wiki/xacro -->
   <xacro:youbot_base name="base"/>
 </robot>

File: youbot_description/urdf/sensors/hokuyo_urg04_laser.gazebo.xacro (robot description, xacro)
@@ -1,10 +1,7 @@
 <?xml version="1.0"?>
-<robot xmlns:sensor="http://playerstage.sourceforge.net/gazebo/xmlschema/#sensor"
-       xmlns:controller="http://playerstage.sourceforge.net/gazebo/xmlschema/#controller"
-       xmlns:interface="http://playerstage.sourceforge.net/gazebo/xmlschema/#interface"
-       xmlns:xacro="http://ros.org/wiki/xacro">
+<robot xmlns:xacro="http://ros.org/wiki/xacro">
   <xacro:macro name="hokuyo_urg04_laser_gazebo" params="name ros_topic update_rate min_angle max_angle">
     <gazebo reference="${name}_link">
-      <sensor name="${name}" type="ray">
+      <sensor name="${name}" type="gpu_ray">
         <pose>0 0 0 0 0 0</pose>
         <ray>
@@ -26,5 +23,5 @@
         <update_rate>${update_rate}</update_rate>
         <visualize>0</visualize>
-        <plugin name="gazebo_ros_laser" filename="libgazebo_ros_laser.so">
+        <plugin name="gazebo_ros_laser" filename="libgazebo_ros_gpu_laser.so">
           <gaussianNoise>0.02</gaussianNoise>
           <alwaysOn>true</alwaysOn>
@@ -33,5 +30,5 @@
           <topicName>${ros_topic}</topicName>
           <frameName>/${name}_link</frameName>
-          <interface:laser name="gazebo_ros_${name}_iface" />
+          <!--interface:laser name="gazebo_ros_${name}_iface" /-->
         </plugin>
       </sensor>

File: youbot_description/urdf/sensors/hokuyo_urg04_laser.urdf.xacro (robot description, xacro)
@@ -1,7 +1,4 @@
 <?xml version="1.0"?>
-<robot xmlns:sensor="http://playerstage.sourceforge.net/gazebo/xmlschema/#sensor"
-       xmlns:controller="http://playerstage.sourceforge.net/gazebo/xmlschema/#controller"
-       xmlns:interface="http://playerstage.sourceforge.net/gazebo/xmlschema/#interface"
-       xmlns:xacro="http://ros.org/wiki/xacro">
+<robot xmlns:xacro="http://ros.org/wiki/xacro">
   <xacro:include filename="$(find youbot_description)/urdf/sensors/hokuyo_urg04_laser.gazebo.xacro" />
   <xacro:macro name="hokuyo_urg04_laser" params="name parent *origin ros_topic update_rate min_angle max_angle">
@@ -23,5 +20,4 @@
 		<mesh filename="package://youbot_description/meshes/sensors/hokuyo.dae" />
 	</geometry>
-	<material name="DarkGrey" />
       </visual>
       <collision>

File: youbot_description/urdf/youbot_arm/arm.urdf.xacro (robot description, xacro)
@@ -1,9 +1,4 @@
 <?xml version="1.0"?>
-<robot  xmlns:sensor="http://playerstage.sourceforge.net/gazebo/xmlschema/#sensor"
-        xmlns:controller="http://playerstage.sourceforge.net/gazebo/xmlschema/#controller"
-        xmlns:interface="http://playerstage.sourceforge.net/gazebo/xmlschema/#interface"
-        xmlns:xacro="http://ros.org/wiki/xacro">
-	<xacro:include filename="$(find youbot_description)/urdf/youbot_arm/arm.gazebo.xacro" />
-	<xacro:include filename="$(find youbot_description)/urdf/youbot_arm/arm.transmission.xacro" />
+<robot  xmlns:xacro="http://ros.org/wiki/xacro">
 	<xacro:include filename="$(find youbot_description)/urdf/youbot_arm/limits.urdf.xacro" />
 	<xacro:macro name="youbot_arm" params="parent name *origin">
@@ -16,5 +11,4 @@
 		<link name="${name}_link_0">
 			<inertial>
-				<!--<origin xyz="0.023 0 0.006" rpy="0 0 0"/>-->
 				<origin xyz="0 0 0" rpy="0 0 0"/>
 				<mass value="${link_0_mass}"/>
@@ -26,12 +20,9 @@
 					<mesh filename="package://youbot_description/meshes/youbot_arm/arm0.dae" />
 				</geometry>
-				<material name="DarkGrey" />
 			</visual>
 			<collision>
-				<!--<origin xyz="0.023 0 0.006" rpy="0 0 0"/>-->
 				<origin xyz="0 0 0" rpy="0 0 0"/>
 				<geometry>
 					<mesh filename="package://youbot_description/meshes/youbot_arm/arm0_convex.dae" />
-					<!--<cylinder length="0.078" radius="0.093"/>-->
 				</geometry>
 			</collision>
@@ -43,15 +34,7 @@
 			<child link="${name}_link_1"/>
 			<axis xyz="0 0 -1"/>
-			<!--<calibration rising="${arm_1_ref}" falling="${arm_1_ref}"/>-->
 			<dynamics damping="1" friction="1" />
-			<!-- damping - N*s/m, N*s*m/rad -->
-			<!-- friction - N, N*m -->
 			<limit effort="${9.5}" velocity="${M_PI / 2.0}" lower="0" upper="${joint_1_limit}"/>
-			<!--effort - N, N*m-->
-			<!--velocity - m/s, rad/s-->
 			<safety_controller k_position="20" k_velocity="${9.5/M_PI / 2.0}" soft_lower_limit="${threshold}" soft_upper_limit="${joint_1_limit_soft}" />
-			<!--k_position N/m, N/rad-->
-			<!--k_velocity N*s/m, N*s*m/rad-->
-			<!--for details: http://www.ros.org/wiki/pr2_controller_manager/safety_limits-->
 		</joint>
 		<link name="${name}_link_1">
@@ -65,12 +48,9 @@
 					<mesh filename="package://youbot_description/meshes/youbot_arm/arm1.dae" />
 				</geometry>
-				<!--<material name="Orange" />-->
 			</visual>
 			<collision>
-				<!--<origin xyz="0 0 -0.003" rpy="0 0 0" />-->
 				<origin xyz="0 0 0" rpy="0 0 0" />
 				<geometry>
 					<mesh filename="package://youbot_description/meshes/youbot_arm/arm1_convex.dae" />
-					<!--<cylinder length="0.102" radius="0.080"/>-->
 				</geometry>
 			</collision>
@@ -82,5 +62,4 @@
 			<child link="${name}_link_2"/>
 			<axis xyz="0 1 0"/>
-			<!--<calibration rising="${arm_2_ref}" falling="${arm_2_ref}"/>-->
 			<dynamics damping="1" friction="1" />
 			<limit effort="${9.5}" velocity="${M_PI / 2.0}" lower="0" upper="${joint_2_limit}"/>
@@ -100,22 +79,11 @@
 			</visual>
 			<collision>
-				<!--<origin xyz="0.001 -0.041 0.074" rpy="0 0 0" />-->
 				<origin xyz="0 -0.032 0.078" rpy="0 0 0" />
 				<geometry>
 					<mesh filename="package://youbot_description/meshes/youbot_arm/arm2_convex.dae" />
-					<!--<box size="0.074 0.082 0.222"/>-->
 				</geometry>
 			</collision>
 		</link>
 		<!-- joint between arm_2_link and arm_3_link -->
-		<!--<joint name="${name}_joint_3" type="revolute">
-			<origin xyz="0.000 0.000 0.155" rpy="0 ${146 * M_PI / 180} 0"/>
-			<parent link="${name}_link_2"/>
-			<child link="${name}_link_3"/>
-			<axis xyz="0 1 0"/>
-			<dynamics damping="1" friction="1" />
-			<limit effort="${6}" velocity="${M_PI / 2.0}" lower="-${joint_3_limit}" upper="0"/>
-                        <safety_controller k_position="20" k_velocity="50" soft_lower_limit="-${joint_3_limit_soft}" soft_upper_limit="${threshold}" />
-		</joint>-->
 		<joint name="${name}_joint_3" type="revolute">
 			<origin xyz="0.000 0.000 0.155" rpy="0 ${146 * M_PI / 180} 0"/>
@@ -140,9 +108,7 @@
 			</visual>
 			<collision>
-				<!--<origin xyz="0.000 0.025 0.067" rpy="0 0 0" />-->
 				<origin xyz="0.000 0.028 0.079" rpy="0 0 0" />
 				<geometry>
 					<mesh filename="package://youbot_description/meshes/youbot_arm/arm3_convex.dae" />
-					<!--<box size="0.064 0.054 0.192"/>-->
 				</geometry>
 			</collision>
@@ -154,5 +120,4 @@
 			<child link="${name}_link_4"/>
 			<axis xyz="0 1 0" />
-			<!--<calibration rising="${arm_4_ref}" falling="${arm_4_ref}"/>-->
 			<dynamics damping="1" friction="1" />
 			<limit effort="${2}" velocity="${M_PI / 2.0}" lower="0" upper="${joint_4_limit}"/>
@@ -172,9 +137,7 @@
 			</visual>
 			<collision>
-				<!--<origin xyz="0 0 0.026" rpy="0 0 0" />-->
 				<origin xyz="0 -0.010 0.029" rpy="0 0 0"/>
 				<geometry>
 					<mesh filename="package://youbot_description/meshes/youbot_arm/arm4_convex.dae" />
-					<!--<box size="0.058 0.100 0.118"/>-->
 				</geometry>
 			</collision>
@@ -186,5 +149,4 @@
 			<child link="${name}_link_5"/>
 			<axis xyz="0 0 -1" />
-			<!--<calibration rising="${arm_5_ref}" falling="${arm_5_ref}"/>-->
 			<dynamics damping="1" friction="1" />
 			<limit effort="1" velocity="${M_PI / 2.0}" lower="0" upper="${joint_5_limit}" />
@@ -207,11 +169,7 @@
 				<geometry>
 					<mesh filename="package://youbot_description/meshes/youbot_arm/arm5_convex.dae" />
-					<!--<box size="0.054 0.096 0.030"/>-->
 				</geometry>
 			</collision>
 		</link>
-		<!-- extensions -->
-		<xacro:youbot_arm_gazebo name="${name}" />
-		<xacro:youbot_arm_transmission name="${name}" />
 	</xacro:macro>
 </robot>

File: youbot_description/urdf/youbot_arm/limits.urdf.xacro (robot description, xacro)
@@ -22,10 +22,4 @@
 	<property name="link_4_mass" value="0.877" />
 	<property name="link_5_mass" value="0.251" />
-	<!--<property name="link_0_mass" value="0.845" />
-	<property name="link_1_mass" value="0.1" />
-	<property name="link_2_mass" value="0.1" />
-	<property name="link_3_mass" value="0.1" />
-	<property name="link_4_mass" value="0.1" />
-	<property name="link_5_mass" value="0.1" />-->
 	<!-- TODO: add inertia tensor-->
 	<xacro:macro name="default_origin">

File: youbot_description/urdf/youbot_base/base.gazebo.xacro (robot description, xacro)
@@ -1,54 +1,14 @@
 <?xml version="1.0"?>
-<robot xmlns:sensor="http://playerstage.sourceforge.net/gazebo/xmlschema/#sensor"
-       xmlns:controller="http://playerstage.sourceforge.net/gazebo/xmlschema/#controller"
-       xmlns:interface="http://playerstage.sourceforge.net/gazebo/xmlschema/#interface"
-       xmlns:xacro="http://ros.org/wiki/xacro">
-	<xacro:macro name="youbot_base_gazebo">
-		<gazebo reference="youbot_base">
-     			<material value="youbot/DarkGrey" />
-    		</gazebo>
-	<!-- front left wheel -->
-    		<gazebo reference="wheel_link_fl">
-       			<material value="youbot/Orange" />
-    		</gazebo>
-    		<gazebo reference="caster_link_fl">
-      			<material value="youbot/Orange" />
-    		</gazebo>
-	<!-- front right wheel -->
-    		<gazebo reference="wheel_link_fr">
-       			<material value="youbot/Orange" />
-    		</gazebo>
-    		<gazebo reference="caster_link_fr">
-      			<material value="youbot/Orange" />
-    		</gazebo>
-	<!-- back left wheel -->
-    		<gazebo reference="wheel_link_bl">
-       			<material value="youbot/Orange" />
-    		</gazebo>
-    		<gazebo reference="caster_link_bl">
-      			<material value="youbot/Orange" />
-    		</gazebo>
-	<!-- back right wheel -->
-    		<gazebo reference="wheel_link_br">
-       			<material value="youbot/Orange" />
-    		</gazebo>
-    		<gazebo reference="caster_link_br">
-      			<material value="youbot/Orange" />
-    		</gazebo>
-	<!-- position controller -->
-		<gazebo>
-      			<plugin name="gazebo_ros_p3d" filename="libgazebo_ros_p3d.so">
-        			<alwaysOn>true</alwaysOn>
-        			<updateRate>100.0</updateRate>
-        			<bodyName>base_link</bodyName>
-        			<topicName>base_pose_ground_truth</topicName>
-        			<gaussianNoise>0.01</gaussianNoise>
-        			<frameName>map</frameName>
-        			<xyzOffsets>25.7 25.7 0</xyzOffsets> <!-- initialize odometry for fake localization-->
-        			<rpyOffsets>0 0 0</rpyOffsets>
-        			<interface:position name="p3d_base_position"/>
-      			</plugin>
-      			<canonicalBody>base_footprint</canonicalBody>
-    		</gazebo>
+<robot xmlns:xacro="http://ros.org/wiki/xacro">
+  <xacro:macro name="youbot_base_controller">
+    <gazebo>
+      <plugin name="base_controller" filename="libyoubot_base_controller.so">
+        <commandTopic>cmd_vel</commandTopic>
+        <odometryTopic>odom</odometryTopic>
+        <odometryFrame>odom</odometryFrame>
+        <odometryRate>20.0</odometryRate>
+        <robotBaseFrame>base_link</robotBaseFrame>
+      </plugin>
+    </gazebo>
   </xacro:macro>
 </robot>
