Commit message: cleaned up youbot description, added meccanum wheels no urdf, added gazebo packages

File: youbot_description/urdf/youbot_base/base.urdf.xacro (robot description, xacro)
@@ -1,15 +1,7 @@
 <?xml version="1.0"?>
-<robot  xmlns:sensor="http://playerstage.sourceforge.net/gazebo/xmlschema/#sensor"
-        xmlns:controller="http://playerstage.sourceforge.net/gazebo/xmlschema/#controller"
-        xmlns:interface="http://playerstage.sourceforge.net/gazebo/xmlschema/#interface"
-        xmlns:xacro="http://ros.org/wiki/xacro">
+<robot  xmlns:xacro="http://ros.org/wiki/xacro">
 	<!-- sensors -->
 	<xacro:include filename="$(find youbot_description)/urdf/sensors/hokuyo_urg04_laser.urdf.xacro"/>
-	<!--include filename="$(find youbot_description)/urdf/sensors/ultrasonicleftfront.urdf.xacro"/>
-	<xacro:include filename="$(find youbot_description)/urdf/sensors/ultrasonicleftback.urdf.xacro"/>
-	<xacro:include filename="$(find youbot_description)/urdf/sensors/ultrasonicrightfront.urdf.xacro"/>
-	<xacro:include filename="$(find youbot_description)/urdf/sensors/ultrasonicrightback.urdf.xacro"/-->
-	<xacro:include filename="$(find youbot_description)/urdf/youbot_base/base.gazebo.xacro" />
-	<xacro:include filename="$(find youbot_description)/urdf/youbot_base/base.transmission.xacro" />
+        <xacro:include filename="$(find youbot_description)/urdf/youbot_base/base.gazebo.xacro" />
  	<!-- simplified box collision geometry for base -->
   	<property name="base_size_x" value="0.570" />
@@ -26,5 +18,5 @@
 	<property name="wheel_mass" value="0.4" />
 	<property name="wheel_radius" value="0.05" />
-	<property name="wheel_length" value="0.005" />
+	<property name="wheel_length" value="0.07" />
 	<property name="caster_joint_damping" value="1.0" />
 	<property name="caster_joint_friction" value="1.0" />
@@ -32,6 +24,6 @@
 	<property name="caster_joint_velocity" value="10" />
 	<property name="caster_joint_safety_k_velocity" value="10.0" />
-	<property name="wheel_joint_damping" value="1.0" />
-	<property name="wheel_joint_friction" value="1.0" />
+	<property name="wheel_joint_damping" value="0.0" />
+	<property name="wheel_joint_friction" value="0.0" />
 	<property name="wheel_joint_effort" value="30" />
 	<property name="wheel_joint_velocity" value="10" />
@@ -39,10 +31,10 @@
 	<xacro:macro name="youbot_base" params="name">
 		<link name="${name}_footprint">
-      			<!--inertial>
-        			<mass value="0.1" />
+      			<inertial>
+        			<mass value="0.01" />
         			<origin xyz="0 0 ${-base_size_z / 2.0}" rpy="0 0 0" />
-        			<inertia ixx="1.0" ixy="0.0" ixz="0.0"
-                 			iyy="1.0" iyz="0.0" izz="1.0" />
-      				</inertial-->
+        			<inertia ixx="0.001" ixy="0.001" ixz="0.001"
+                 			iyy="0.001" iyz="0.001" izz="0.001" />
+      			</inertial>
       			<visual>
         			<origin xyz="0 0 0" rpy="0 0 0" />
@@ -81,27 +73,10 @@
         			<origin xyz="0 0 0" rpy="0 0 0" />
         			<geometry>
-          				<!--<box size="${base_size_x} ${base_size_y} ${base_size_z}" />-->
 					<mesh filename="package://youbot_description/meshes/youbot_base/base_convex.dae"/>
 	       			</geometry>
       			</collision>
     		</link>
-<!-- links vorne -->
-    		<xacro:ultrasonicleftfront_laser name="ultrasonic_frame_0" parent="${name}" ros_topic="ultrasonic_scan_0" update_rate="10" min_angle="${-M_PI/8}" max_angle="${M_PI/8}" >
-     			 <origin xyz="0.08 0.18 -0.067" rpy="0 0 ${M_PI/2}" />
-    		</xacro:ultrasonicleftfront_laser>
-<!-- links hinten -->
-    		<xacro:ultrasonicleftback_laser name="ultrasonic_frame_1" parent="${name}" ros_topic="ultrasonic_scan_1" update_rate="10" min_angle="${-M_PI/8}" max_angle="${M_PI/8}" >
-     			 <origin xyz="-0.08 0.18 -0.067" rpy="0 0 ${M_PI/2}" />
-    		</xacro:ultrasonicleftback_laser>
-<!-- rechts vorne -->
-    		<xacro:ultrasonicrightfront_laser name="ultrasonic_frame_2" parent="${name}" ros_topic="ultrasonic_scan_2" update_rate="10" min_angle="${-M_PI/8}" max_angle="${M_PI/8}" >
-     			 <origin xyz="0.08 -0.18 -0.067" rpy="0 0 ${-M_PI/2}" />
-    		</xacro:ultrasonicrightfront_laser>
-<!-- rechts hinten -->
-    		<xacro:ultrasonicrightback_laser name="ultrasonic_frame_3" parent="${name}" ros_topic="ultrasonic_scan_3" update_rate="10" min_angle="${-M_PI/8}" max_angle="${+M_PI/8}" >
-     			 <origin xyz="-0.08 -0.18 -0.067" rpy="0 0 ${-M_PI/2}" />
-    		</xacro:ultrasonicrightback_laser>
 		<!-- base laser front -->
-    		<xacro:hokuyo_urg04_laser name="${name}_laser_front" parent="${name}" ros_topic="scan_front" update_rate="10" min_angle="-1.57" max_angle="1.57" >
+    		<xacro:hokuyo_urg04_laser name="${name}_laser_front" parent="${name}" ros_topic="scan" update_rate="10" min_angle="-1.57" max_angle="1.57" >
      			 <origin xyz="0.309 0 -0.03" rpy="0 0 0" />
     		</xacro:hokuyo_urg04_laser>
@@ -110,31 +85,14 @@
      			 <origin xyz="-0.309 0 -0.03" rpy="0 0 ${M_PI}" />
     		</xacro:hokuyo_urg04_laser>
-	<!-- front left wheel -->
-		<joint name="caster_joint_fl" type="continuous">
+	        <!-- front left wheel -->
+		<joint name="wheel_joint_fl" type="continuous">
 			<origin xyz="${caster_offset_x} ${caster_offset_y} ${caster_offset_z}" rpy="0 0 0" />
-      			<axis xyz="0 0 1" />
-      			<limit effort="${caster_joint_effort}" velocity="${caster_joint_velocity}"/>
-      			<dynamics damping="${caster_joint_damping}" friction="${caster_joint_friction}" />
-			<safety_controller k_velocity="${caster_joint_safety_k_velocity}" />
-			<parent link="${name}_link"/>
-      			<child link="caster_link_fl" />
-    		</joint>
-		<link name="caster_link_fl">
-      			<inertial>
-        			<mass value="${caster_mass}" />
-        			<origin xyz="0 0 0" />
-        			<inertia  ixx="0.012411765597" ixy="-0.000711733678" ixz="0.00050272983"
-                  			iyy="0.015218160428" iyz="-0.000004273467" izz="0.011763977943" />
-      			</inertial>
-   		</link>
-		<joint name="wheel_joint_fl" type="continuous">
-      			<axis xyz="0 1 0" />
-      			<limit effort="${wheel_joint_effort}" velocity="${wheel_joint_velocity}"/>
-            		<origin xyz="${wheel_offset_x} ${wheel_offset_y} ${wheel_offset_z}" rpy="0 0 0" />
-      			<parent link="caster_link_fl"/>
-			<dynamics damping="${wheel_joint_damping}" friction="${wheel_joint_friction}" />
-			<safety_controller k_velocity="${wheel_joint_safety_k_velocity}" />
-      			<child link="wheel_link_fl"/>
-     		</joint>
+      			<axis xyz="0 1 0" />
+      			<limit effort="${caster_joint_effort}" velocity="${caster_joint_velocity}"/>
+      			<dynamics damping="${caster_joint_damping}" friction="${caster_joint_friction}" />
+			<safety_controller k_velocity="${caster_joint_safety_k_velocity}" />
+			<parent link="${name}_link"/>
+      			<child link="wheel_link_fl" />
+    		</joint>
     		<link name="wheel_link_fl">
       			<inertial>
@@ -146,45 +104,56 @@
       			<visual>
         			<origin xyz="0 0 0" rpy="0 0 0" />
-					<!--<mesh filename="package://youbot_description/meshes/youbot_base/youbot_wheel.stl" />-->
+                                <geometry>
+				        <mesh filename="package://youbot_description/meshes/youbot_base/wheel1.dae" />
+                                </geometry>
+      			</visual>
+      			<collision>
+        			<origin xyz="0 0 0" rpy="${M_PI/2} 0 0" />
+        			<geometry>
+        		       		<cylinder radius="${wheel_radius}" length="${wheel_length}"/>
+        	       		</geometry>
+      			</collision>
+    		</link>
+	<!-- front right wheel -->
+		<joint name="wheel_joint_fr" type="continuous">
+			<origin xyz="${caster_offset_x} ${-caster_offset_y} ${caster_offset_z}" rpy="0 0 0" />
+      			<axis xyz="0 1 0" />
+      			<limit effort="${caster_joint_effort}" velocity="${caster_joint_velocity}"/>
+      			<dynamics damping="${caster_joint_damping}" friction="${caster_joint_friction}" />
+			<safety_controller k_velocity="${caster_joint_safety_k_velocity}" />
+			<parent link="${name}_link"/>
+      			<child link="wheel_link_fr" />
+    		</joint>
+    		<link name="wheel_link_fr">
+      			<inertial>
+        		<mass value="${wheel_mass}" />
+        		<origin xyz="0 0 0" />
+       			<inertia  ixx="0.012411765597" ixy="-0.000711733678" ixz="0.00050272983"
+                  		iyy="0.015218160428" iyz="-0.000004273467" izz="0.011763977943" />
+      			</inertial>
+      			<visual>
+        			<origin xyz="0 0 0" rpy="0 0 0" />
 				<geometry>
-					<sphere radius="${wheel_radius}"/>
-				</geometry>
-       				<material name="Orange" />
-      			</visual>
-      			<collision>
-        			<origin xyz="0 0 0" rpy="${M_PI/2} 0 0" />
-        			<geometry>
-        		       		<cylinder radius="${wheel_radius}" length="${wheel_radius}" />
-        	       		</geometry>
-      			</collision>
-    		</link>
-	<!-- front right wheel -->
-		<joint name="caster_joint_fr" type="continuous">
-			<origin xyz="${caster_offset_x} ${-caster_offset_y} ${caster_offset_z}" rpy="0 0 0" />
-      			<axis xyz="0 0 1" />
-      			<limit effort="${caster_joint_effort}" velocity="${caster_joint_velocity}"/>
-      			<dynamics damping="${caster_joint_damping}" friction="${caster_joint_friction}" />
-			<safety_controller k_velocity="${caster_joint_safety_k_velocity}" />
-			<parent link="${name}_link"/>
-      			<child link="caster_link_fr" />
-    		</joint>
-		<link name="caster_link_fr">
-      			<inertial>
-        			<mass value="${caster_mass}" />
-        			<origin xyz="0 0 0" />
-        			<inertia  ixx="0.012411765597" ixy="-0.000711733678" ixz="0.00050272983"
-                  			iyy="0.015218160428" iyz="-0.000004273467" izz="0.011763977943" />
-      				</inertial>
-   		</link>
-		<joint name="wheel_joint_fr" type="continuous">
-      			<axis xyz="0 1 0" />
-      			<limit effort="${wheel_joint_effort}" velocity="${wheel_joint_velocity}"/>
-            		<dynamics damping="${wheel_joint_damping}" friction="${wheel_joint_friction}" />
-			<safety_controller k_velocity="${wheel_joint_safety_k_velocity}" />
-      			<origin xyz="${wheel_offset_x} ${wheel_offset_y} ${wheel_offset_z}" rpy="0 0 0" />
-      			<parent link="caster_link_fr"/>
-      			<child link="wheel_link_fr"/>
-     		</joint>
-    		<link name="wheel_link_fr">
+          				<mesh filename="package://youbot_description/meshes/youbot_base/wheel2.dae" />
+        			</geometry>
+      			</visual>
+      			<collision>
+        			<origin xyz="0 0 0" rpy="${M_PI/2} 0 0" />
+        			<geometry>
+        		       		<cylinder radius="${wheel_radius}" length="${wheel_length}"/>
+        	       		</geometry>
+      			</collision>
+    		</link>
+	        <!-- back left wheel -->
+		<joint name="wheel_joint_bl" type="continuous">
+			<origin xyz="${-caster_offset_x} ${caster_offset_y} ${caster_offset_z}" rpy="0 0 0" />
+      			<axis xyz="0 1 0" />
+      			<limit effort="${caster_joint_effort}" velocity="${caster_joint_velocity}"/>
+      			<dynamics damping="${caster_joint_damping}" friction="${caster_joint_friction}" />
+			<safety_controller k_velocity="${caster_joint_safety_k_velocity}" />
+			<parent link="${name}_link"/>
+      			<child link="wheel_link_bl" />
+    		</joint>
+    		<link name="wheel_link_bl">
       			<inertial>
         		<mass value="${wheel_mass}" />
@@ -196,45 +165,25 @@
         			<origin xyz="0 0 0" rpy="0 0 0" />
 				<geometry>
-          				<!--<mesh filename="package://youbot_description/meshes/youbot_base/youbot_wheel.stl" />-->
-					<sphere radius="${wheel_radius}"/>
-        			</geometry>
-       				<material name="Orange" />
-      			</visual>
-      			<collision>
-        			<origin xyz="0 0 0" rpy="${M_PI/2} 0 0" />
-        			<geometry>
-        		       		<cylinder radius="${wheel_radius}" length="${wheel_radius}" />
-        	       		</geometry>
-      			</collision>
-    		</link>
-	<!-- back left wheel -->
-		<joint name="caster_joint_bl" type="continuous">
-			<origin xyz="${-caster_offset_x} ${caster_offset_y} ${caster_offset_z}" rpy="0 0 0" />
-      			<axis xyz="0 0 1" />
-      			<limit effort="${caster_joint_effort}" velocity="${caster_joint_velocity}"/>
-      			<dynamics damping="${caster_joint_damping}" friction="${caster_joint_friction}" />
-			<safety_controller k_velocity="${caster_joint_safety_k_velocity}" />
-			<parent link="${name}_link"/>
-      			<child link="caster_link_bl" />
-    		</joint>
-		<link name="caster_link_bl">
-      			<inertial>
-        			<mass value="${caster_mass}" />
-        			<origin xyz="0 0 0" />
-        			<inertia  ixx="0.012411765597" ixy="-0.000711733678" ixz="0.00050272983"
-                  			iyy="0.015218160428" iyz="-0.000004273467" izz="0.011763977943" />
-      				</inertial>
-   		</link>
-		<joint name="wheel_joint_bl" type="continuous">
-      			<axis xyz="0 1 0" />
-      			<limit effort="10" velocity="10"/>
-			<limit effort="${wheel_joint_effort}" velocity="${wheel_joint_velocity}"/>
-			<dynamics damping="${wheel_joint_damping}" friction="${wheel_joint_friction}" />
-			<safety_controller k_velocity="${wheel_joint_safety_k_velocity}" />
-      			<origin xyz="${wheel_offset_x} ${wheel_offset_y} ${wheel_offset_z}" rpy="0 0 0" />
-      			<parent link="caster_link_bl"/>
-      			<child link="wheel_link_bl"/>
-     		</joint>
-    		<link name="wheel_link_bl">
+          				<mesh filename="package://youbot_description/meshes/youbot_base/wheel2.dae" />
+        			</geometry>
+      			</visual>
+      			<collision>
+        			<origin xyz="0 0 0" rpy="${M_PI/2} 0 0" />
+        			<geometry>
+        		       		<cylinder radius="${wheel_radius}" length="${wheel_length}"/>
+        	       		</geometry>
+      			</collision>
+    		</link>
+	<!-- back right wheel -->
+		<joint name="wheel_joint_br" type="continuous">
+			<origin xyz="${-caster_offset_x} ${-caster_offset_y} ${caster_offset_z}" rpy="0 0 0" />
+      			<axis xyz="0 1 0" />
+      			<limit effort="${caster_joint_effort}" velocity="${caster_joint_velocity}"/>
+      			<dynamics damping="${caster_joint_damping}" friction="${caster_joint_friction}" />
+			<safety_controller k_velocity="${caster_joint_safety_k_velocity}" />
+			<parent link="${name}_link"/>
+      			<child link="wheel_link_br" />
+    		</joint>
+    		<link name="wheel_link_br">
       			<inertial>
         		<mass value="${wheel_mass}" />
@@ -246,68 +195,15 @@
         			<origin xyz="0 0 0" rpy="0 0 0" />
 				<geometry>
-          				<!--<mesh filename="package://youbot_description/meshes/youbot_base/youbot_wheel.stl" />-->
-					<sphere radius="${wheel_radius}"/>
-        			</geometry>
-       				<material name="Orange" />
-      			</visual>
-      			<collision>
-        			<origin xyz="0 0 0" rpy="${M_PI/2} 0 0" />
-        			<geometry>
-        		       		<cylinder radius="${wheel_radius}" length="${wheel_radius}" />
-        	       		</geometry>
-      			</collision>
-    		</link>
-	<!-- back right wheel -->
-		<joint name="caster_joint_br" type="continuous">
-			<origin xyz="${-caster_offset_x} ${-caster_offset_y} ${caster_offset_z}" rpy="0 0 0" />
-      			<axis xyz="0 0 1" />
-      			<limit effort="${caster_joint_effort}" velocity="${caster_joint_velocity}"/>
-      			<dynamics damping="${caster_joint_damping}" friction="${caster_joint_friction}" />
-			<safety_controller k_velocity="${caster_joint_safety_k_velocity}" />
-			<parent link="${name}_link"/>
-      			<child link="caster_link_br" />
-    		</joint>
-		<link name="caster_link_br">
-      			<inertial>
-        			<mass value="${caster_mass}" />
-        			<origin xyz="0 0 0" />
-        			<inertia  ixx="0.012411765597" ixy="-0.000711733678" ixz="0.00050272983"
-                  			iyy="0.015218160428" iyz="-0.000004273467" izz="0.011763977943" />
-      				</inertial>
-   		</link>
-		<joint name="wheel_joint_br" type="continuous">
-      			<axis xyz="0 1 0" />
-      			<limit effort="${wheel_joint_effort}" velocity="${wheel_joint_velocity}"/>
-            		<dynamics damping="${wheel_joint_damping}" friction="${wheel_joint_friction}" />
-			<safety_controller k_velocity="${wheel_joint_safety_k_velocity}" />
-      			<origin xyz="${wheel_offset_x} ${wheel_offset_y} ${wheel_offset_z}" rpy="0 0 0" />
-      			<parent link="caster_link_br"/>
-      			<child link="wheel_link_br"/>
-     		</joint>
-    		<link name="wheel_link_br">
-      			<inertial>
-        		<mass value="${wheel_mass}" />
-        		<origin xyz="0 0 0" />
-       			<inertia  ixx="0.012411765597" ixy="-0.000711733678" ixz="0.00050272983"
-                  		iyy="0.015218160428" iyz="-0.000004273467" izz="0.011763977943" />
-      			</inertial>
-      			<visual>
-        			<origin xyz="0 0 0" rpy="0 0 0" />
-				<geometry>
-          				<!--<mesh filename="package://youbot_description/meshes/youbot_base/youbot_wheel.stl" />-->
-					<sphere radius="${wheel_radius}"/>
-        			</geometry>
-       				<material name="Orange" />
-      			</visual>
-      			<collision>
-        			<origin xyz="0 0 0" rpy="${M_PI/2} 0 0" />
-        			<geometry>
-        		       		<cylinder radius="${wheel_radius}" length="${wheel_radius}" />
-        	       		</geometry>
-      			</collision>
-    		</link>
-	<!-- extensions -->
-		<xacro:youbot_base_gazebo />
-		<xacro:youbot_base_transmission />
+          				<mesh filename="package://youbot_description/meshes/youbot_base/wheel1.dae" />
+        			</geometry>
+      			</visual>
+      			<collision>
+        			<origin xyz="0 0 0" rpy="${M_PI/2} 0 0" />
+        			<geometry>
+        		       		<cylinder radius="${wheel_radius}" length="${wheel_length}"/>
+        	       		</geometry>
+      			</collision>
+    		</link>
+                <xacro:youbot_base_controller/>
 	</xacro:macro>
 </robot>

File: youbot_description/urdf/youbot_gripper/gripper.urdf.xacro (robot description, xacro)
@@ -1,9 +1,4 @@
 <?xml version="1.0"?>
-<robot xmlns:sensor="http://playerstage.sourceforge.net/gazebo/xmlschema/#sensor"
-       xmlns:controller="http://playerstage.sourceforge.net/gazebo/xmlschema/#controller"
-       xmlns:interface="http://playerstage.sourceforge.net/gazebo/xmlschema/#interface"
-       xmlns:xacro="http://ros.org/wiki/xacro">
-	<xacro:include filename="$(find youbot_description)/urdf/youbot_gripper/gripper.gazebo.xacro" />
-	<xacro:include filename="$(find youbot_description)/urdf/youbot_gripper/gripper.transmission.xacro" />
+<robot xmlns:xacro="http://ros.org/wiki/xacro">
 	<xacro:include filename="$(find youbot_description)/urdf/youbot_gripper/limits.urdf.xacro" />
 	<xacro:macro name="youbot_gripper" params="parent name *origin">
@@ -25,11 +20,9 @@
 					<mesh filename="package://youbot_description/meshes/youbot_gripper/palm.dae" />
 				</geometry>
-				<material name="Black" />
 			</visual>
 			<collision>
 				<origin xyz="0.003 0 0.01" rpy="0 0 0" />
 				<geometry>
-					<box size="0.05 0.09 0.065"/>
-					<!--<mesh filename="package://youbot_description/meshes/youbot_gripper/palm.STL" />-->
+					<mesh filename="package://youbot_description/meshes/youbot_gripper/palm_convex.dae" />
 				</geometry>
 			</collision>
@@ -53,6 +46,5 @@
 				<origin xyz="0.0078 0 -0.0144" rpy="0 ${-M_PI/2} 0" /> <!---->
 				<geometry>
-					<!--<box size="0.014 0.020 0.068"/>-->
-					<mesh filename="package://youbot_description/meshes/youbot_gripper/finger.STL" />
+					<mesh filename="package://youbot_description/meshes/youbot_gripper/finger.dae" />
 				</geometry>
 				<material name="DarkGrey" />
@@ -61,6 +53,5 @@
 				<origin xyz="0.0007 0.0105 0.0185" rpy="0 0 0" />
 				<geometry>
-					<box size="0.014 0.020 0.068"/>
-					<!--<mesh filename="package://youbot_description/meshes/youbot_gripper/finger.STL" />-->
+					<mesh filename="package://youbot_description/meshes/youbot_gripper/finger_convex.dae" />
 				</geometry>
 			</collision>
@@ -84,6 +75,5 @@
 				<origin xyz="0.0077 0 -0.0144" rpy="0 ${-M_PI/2} 0" /> <!-- -->
 				<geometry>
-					<!--<box size="0.014 0.020 0.068"/>-->
-					<mesh filename="package://youbot_description/meshes/youbot_gripper/finger.STL" />
+					<mesh filename="package://youbot_description/meshes/youbot_gripper/finger.dae" />
 				</geometry>
 				<material name="DarkGrey" />
@@ -92,6 +82,5 @@
 				<origin xyz="0.0007 0.0105 0.0185" rpy="0 0 0" />
 				<geometry>
-					<box size="0.014 0.020 0.068"/>
-					<!--<mesh filename="package://youbot_description/meshes/youbot_gripper/finger.STL" />-->
+					<mesh filename="package://youbot_description/meshes/youbot_gripper/finger_convex.dae" />
 				</geometry>
 			</collision>
@@ -110,22 +99,4 @@
 			</inertial>
 		</link>
-		<!-- coordinate frame for usb_cam from hand-eye-calib -->
-		<joint name="usb_cam_joint" type="fixed">
-			<origin xyz="-0.0417 -0.0078 0.0207" rpy="1.49224 3.09978 1.5769" />
-			<!--<origin xyz="-0.0928 -0.0117 0.0431" rpy="1.50579 2.83312 1.6295" />-->
-			<!--<origin xyz="-0.02476 -0.0244 0.0125" rpy="2.67678 3.15999 3.05878" /> -->
-			<parent link="${name}_tip" />
-			<child link="usb_cam" />
-		</joint>
-		<link name="usb_cam">
-			<inertial>
-				<mass value="0.001" />
-				<origin xyz="0 0 0" />
-				<inertia ixx="0.001" ixy="0.0" ixz="0.0" iyy="0.001" iyz="0.0" izz="0.001" />
-			</inertial>
-		</link>
-		<!-- extensions -->
-		<xacro:youbot_gripper_gazebo name="${name}" />
-		<xacro:youbot_gripper_transmission name="${name}" />
 	</xacro:macro>
 </robot>
