Commit message: added gazebo arm controller and adapted driver node to new urdf

File: youbot_description/robots/youbot.urdf.xacro (robot description, xacro)
@@ -12,4 +12,6 @@
   <!-- youbot gripper -->
   <xacro:include filename="$(find youbot_description)/urdf/youbot_gripper/gripper.urdf.xacro" />
+  <!-- joint state publisher -->
+  <xacro:include filename="$(find youbot_description)/robots/youbot_gazebo.xacro" />
   <!-- Now we can start using the macros included above to define the actual youbot -->
   <xacro:youbot_base name="base"/>
@@ -23,3 +25,4 @@
     <origin xyz="0 0 0" rpy="0 0 0" />
   </xacro:youbot_gripper>
+  <xacro:joint_state_publisher />
 </robot>

File: youbot_description/robots/youbot_base.urdf.xacro (robot description, xacro)
@@ -6,5 +6,8 @@
   <!-- youbot base -->
   <xacro:include filename="$(find youbot_description)/urdf/youbot_base/base.urdf.xacro" />
+  <!-- joint state publisher -->
+  <xacro:include filename="$(find youbot_description)/robots/youbot_gazebo.xacro" />
   <!-- Now we can start using the macros included above to define the actual youbot -->
   <xacro:youbot_base name="base"/>
+  <xacro:joint_state_publisher />
 </robot>

File: youbot_description/urdf/sensors/hokuyo_urg04_laser.gazebo.xacro (robot description, xacro)
@@ -3,5 +3,5 @@
   <xacro:macro name="hokuyo_urg04_laser_gazebo" params="name ros_topic update_rate min_angle max_angle">
     <gazebo reference="${name}_link">
-      <sensor name="${name}" type="gpu_ray">
+      <sensor name="${name}" type="ray">
         <pose>0 0 0 0 0 0</pose>
         <ray>
@@ -20,8 +20,8 @@
           </range>
         </ray>
-        <always_on>0</always_on>
+        <always_on>true</always_on>
         <update_rate>${update_rate}</update_rate>
-        <visualize>0</visualize>
-        <plugin name="gazebo_ros_laser" filename="libgazebo_ros_gpu_laser.so">
+        <visualize>false</visualize>
+        <plugin name="gazebo_ros_laser" filename="libgazebo_ros_laser.so">
           <gaussianNoise>0.02</gaussianNoise>
           <alwaysOn>true</alwaysOn>

File: youbot_description/urdf/youbot_arm/arm.urdf.xacro (robot description, xacro)
@@ -2,4 +2,5 @@
 <robot  xmlns:xacro="http://ros.org/wiki/xacro">
 	<xacro:include filename="$(find youbot_description)/urdf/youbot_arm/limits.urdf.xacro" />
+	<xacro:include filename="$(find youbot_description)/urdf/youbot_arm/arm.gazebo.xacro" />
 	<xacro:macro name="youbot_arm" params="parent name *origin">
 		<!-- joint between base_link and arm_0_link -->
@@ -172,4 +173,5 @@
 			</collision>
 		</link>
+                <xacro:youbot_arm_controller />
 	</xacro:macro>
 </robot>

File: youbot_description/urdf/youbot_base/base.gazebo.xacro (robot description, xacro)
@@ -8,7 +8,7 @@
         <odometryFrame>odom</odometryFrame>
         <odometryRate>20.0</odometryRate>
-        <robotBaseFrame>base_link</robotBaseFrame>
+        <robotBaseFrame>base_footprint</robotBaseFrame>
       </plugin>
-    </gazebo>
+   </gazebo>
   </xacro:macro>
 </robot>

File: youbot_description/urdf/youbot_base/base.urdf.xacro (robot description, xacro)
@@ -9,19 +9,10 @@
   	<property name="base_size_z" value="0.100" />
 	<property name="base_mass" value="22.0" />
-	<property name="caster_offset_x" value="0.228"  />
-  	<property name="caster_offset_y" value="0.158"  />
-  	<property name="caster_offset_z" value="-0.034" />
-	<property name="caster_mass" value="0.1" />
-	<property name="wheel_offset_x" value="0.0"  />
-  	<property name="wheel_offset_y" value="0.0"  />
-  	<property name="wheel_offset_z" value="0.0" />
+	<property name="wheel_offset_x" value="0.228"  />
+  	<property name="wheel_offset_y" value="0.158"  />
+  	<property name="wheel_offset_z" value="-0.034" />
 	<property name="wheel_mass" value="0.4" />
 	<property name="wheel_radius" value="0.05" />
 	<property name="wheel_length" value="0.07" />
-	<property name="caster_joint_damping" value="1.0" />
-	<property name="caster_joint_friction" value="1.0" />
-	<property name="caster_joint_effort" value="30" />
-	<property name="caster_joint_velocity" value="10" />
-	<property name="caster_joint_safety_k_velocity" value="10.0" />
 	<property name="wheel_joint_damping" value="0.0" />
 	<property name="wheel_joint_friction" value="0.0" />
@@ -31,10 +22,4 @@
 	<xacro:macro name="youbot_base" params="name">
 		<link name="${name}_footprint">
-      			<inertial>
-        			<mass value="0.01" />
-        			<origin xyz="0 0 ${-base_size_z / 2.0}" rpy="0 0 0" />
-        			<inertia ixx="0.001" ixy="0.001" ixz="0.001"
-                 			iyy="0.001" iyz="0.001" izz="0.001" />
-      			</inertial>
       			<visual>
         			<origin xyz="0 0 0" rpy="0 0 0" />
@@ -87,9 +72,9 @@
 	        <!-- front left wheel -->
 		<joint name="wheel_joint_fl" type="continuous">
-			<origin xyz="${caster_offset_x} ${caster_offset_y} ${caster_offset_z}" rpy="0 0 0" />
+			<origin xyz="${wheel_offset_x} ${wheel_offset_y} ${wheel_offset_z}" rpy="0 0 0" />
       			<axis xyz="0 1 0" />
-      			<limit effort="${caster_joint_effort}" velocity="${caster_joint_velocity}"/>
-      			<dynamics damping="${caster_joint_damping}" friction="${caster_joint_friction}" />
-			<safety_controller k_velocity="${caster_joint_safety_k_velocity}" />
+      			<limit effort="${wheel_joint_effort}" velocity="${wheel_joint_velocity}"/>
+      			<dynamics damping="${wheel_joint_damping}" friction="${wheel_joint_friction}" />
+			<safety_controller k_velocity="${wheel_joint_safety_k_velocity}" />
 			<parent link="${name}_link"/>
       			<child link="wheel_link_fl" />
@@ -117,9 +102,9 @@
 	<!-- front right wheel -->
 		<joint name="wheel_joint_fr" type="continuous">
-			<origin xyz="${caster_offset_x} ${-caster_offset_y} ${caster_offset_z}" rpy="0 0 0" />
+			<origin xyz="${wheel_offset_x} ${-wheel_offset_y} ${wheel_offset_z}" rpy="0 0 0" />
       			<axis xyz="0 1 0" />
-      			<limit effort="${caster_joint_effort}" velocity="${caster_joint_velocity}"/>
-      			<dynamics damping="${caster_joint_damping}" friction="${caster_joint_friction}" />
-			<safety_controller k_velocity="${caster_joint_safety_k_velocity}" />
+      			<limit effort="${wheel_joint_effort}" velocity="${wheel_joint_velocity}"/>
+      			<dynamics damping="${wheel_joint_damping}" friction="${wheel_joint_friction}" />
+			<safety_controller k_velocity="${wheel_joint_safety_k_velocity}" />
 			<parent link="${name}_link"/>
       			<child link="wheel_link_fr" />
@@ -147,9 +132,9 @@
 	        <!-- back left wheel -->
 		<joint name="wheel_joint_bl" type="continuous">
-			<origin xyz="${-caster_offset_x} ${caster_offset_y} ${caster_offset_z}" rpy="0 0 0" />
+			<origin xyz="${-wheel_offset_x} ${wheel_offset_y} ${wheel_offset_z}" rpy="0 0 0" />
       			<axis xyz="0 1 0" />
-      			<limit effort="${caster_joint_effort}" velocity="${caster_joint_velocity}"/>
-      			<dynamics damping="${caster_joint_damping}" friction="${caster_joint_friction}" />
-			<safety_controller k_velocity="${caster_joint_safety_k_velocity}" />
+      			<limit effort="${wheel_joint_effort}" velocity="${wheel_joint_velocity}"/>
+      			<dynamics damping="${wheel_joint_damping}" friction="${wheel_joint_friction}" />
+			<safety_controller k_velocity="${wheel_joint_safety_k_velocity}" />
 			<parent link="${name}_link"/>
       			<child link="wheel_link_bl" />
@@ -177,9 +162,9 @@
 	<!-- back right wheel -->
 		<joint name="wheel_joint_br" type="continuous">
-			<origin xyz="${-caster_offset_x} ${-caster_offset_y} ${caster_offset_z}" rpy="0 0 0" />
+			<origin xyz="${-wheel_offset_x} ${-wheel_offset_y} ${wheel_offset_z}" rpy="0 0 0" />
       			<axis xyz="0 1 0" />
-      			<limit effort="${caster_joint_effort}" velocity="${caster_joint_velocity}"/>
-      			<dynamics damping="${caster_joint_damping}" friction="${caster_joint_friction}" />
-			<safety_controller k_velocity="${caster_joint_safety_k_velocity}" />
+      			<limit effort="${wheel_joint_effort}" velocity="${wheel_joint_velocity}"/>
+      			<dynamics damping="${wheel_joint_damping}" friction="${wheel_joint_friction}" />
+			<safety_controller k_velocity="${wheel_joint_safety_k_velocity}" />
 			<parent link="${name}_link"/>
       			<child link="wheel_link_br" />

File: youbot_description/urdf/youbot_gripper/gripper.urdf.xacro (robot description, xacro)
@@ -21,10 +21,10 @@
 				</geometry>
 			</visual>
-			<collision>
+			<!--collision>
 				<origin xyz="0.003 0 0.01" rpy="0 0 0" />
 				<geometry>
 					<mesh filename="package://youbot_description/meshes/youbot_gripper/palm_convex.dae" />
 				</geometry>
-			</collision>
+			</collision-->
 		</link>
 		<joint name="${name}_finger_joint_l" type="prismatic">
@@ -44,12 +44,11 @@
 			</inertial>
 			<visual>
-				<origin xyz="0.0078 0 -0.0144" rpy="0 ${-M_PI/2} 0" /> <!---->
+				<origin xyz="0 -0.015 -0.02" rpy="0 ${-M_PI/2} 0" /> <!---->
 				<geometry>
 					<mesh filename="package://youbot_description/meshes/youbot_gripper/finger.dae" />
 				</geometry>
-				<material name="DarkGrey" />
 			</visual>
 			<collision>
-				<origin xyz="0.0007 0.0105 0.0185" rpy="0 0 0" />
+				<origin xyz="0 -0.015 -0.02" rpy="0 ${-M_PI/2} 0" />
 				<geometry>
 					<mesh filename="package://youbot_description/meshes/youbot_gripper/finger_convex.dae" />
@@ -73,12 +72,11 @@
 			</inertial>
 			<visual>
-				<origin xyz="0.0077 0 -0.0144" rpy="0 ${-M_PI/2} 0" /> <!-- -->
+				<origin xyz="0 -0.015 -0.02" rpy="0 ${-M_PI/2} 0" /> <!-- -->
 				<geometry>
 					<mesh filename="package://youbot_description/meshes/youbot_gripper/finger.dae" />
 				</geometry>
-				<material name="DarkGrey" />
 			</visual>
 			<collision>
-				<origin xyz="0.0007 0.0105 0.0185" rpy="0 0 0" />
+				<origin xyz="0 -0.015 -0.02" rpy="0 ${-M_PI/2} 0" />
 				<geometry>
 					<mesh filename="package://youbot_description/meshes/youbot_gripper/finger_convex.dae" />
