Commit message: new launch file striukture

File: luh_youbot_description/urdf/sensors/asus_xtion_camera.urdf.xacro (robot description, xacro)
@@ -7,5 +7,5 @@
 	<link name="${parent}_${suffix}_frame">
 	  <inertial>
-		<mass value="0.01" />
+		<mass value="0.0001" />
 		<origin xyz="0 0 0" />
 		<inertia ixx="0.1" ixy="0" ixz="0" iyy="0.1" iyz="0" izz="0.1" />
@@ -21,5 +21,5 @@
   	<link name="${name}_foot_link">
       <inertial>
-        <mass value="0.05" />
+        <mass value="0.0005" />
         <origin xyz="0 0 0" rpy="0 0 0"/>
         <inertia ixx="0.0001" ixy="0" ixz="0" iyy="0.0001" iyz="0" izz="0.0001" />
@@ -46,5 +46,5 @@
     <link name="${name}_tilt_link">
       <inertial>
-        <mass value="0.01" />
+        <mass value="0.0001" />
         <origin xyz="0 0 0" rpy="0 0 0"/>
         <inertia ixx="0.0001" ixy="0" ixz="0" iyy="0.0001" iyz="0" izz="0.0001" />
@@ -74,5 +74,5 @@
     <link name="${name}_camera">
       <inertial>
-        <mass value="0.1" />
+        <mass value="0.001" />
         <origin xyz="0 0 0" rpy="0 0 0"/>
         <inertia ixx="0.0001" ixy="0" ixz="0" iyy="0.0001" iyz="0" izz="0.0001" />
