Commit message: put new gripper in urdf and added a simple gripper controller for gazebo

File: luh_youbot_description/robots/youbot.urdf.xacro (robot description, xacro)
@@ -15,14 +15,14 @@
   <xacro:include filename="$(find luh_youbot_description)/robots/youbot_gazebo.xacro" />
   <!-- Now we can start using the macros included above to define the actual youbot -->
-  <xacro:youbot_base name="base"/>
+  <xacro:youbot_base name="base" namespace="gazebo"/>
   <xacro:youbot_plate name="plate" parent="base_link">
     <origin xyz="-0.039 0 0.064" rpy="0 0 0" />
   </xacro:youbot_plate>
-  <xacro:youbot_arm name="arm" parent="base_link">
+  <xacro:youbot_arm name="arm" parent="base_link" namespace="gazebo">
     <origin xyz="0.258 0 0.066" rpy="0 0 0.576" />
   </xacro:youbot_arm>
-  <xacro:youbot_gripper name="gripper" parent="arm_link_5">
+  <xacro:youbot_gripper name="gripper" parent="arm_link_5" namespace="">
     <origin xyz="0 0 0" rpy="0 0 0" />
   </xacro:youbot_gripper>
-  <xacro:joint_state_publisher />
+  <xacro:joint_state_publisher namespace="gazebo"/>
 </robot>

File: luh_youbot_description/robots/youbot_base.urdf.xacro (robot description, xacro)
@@ -9,5 +9,5 @@
   <xacro:include filename="$(find luh_youbot_description)/robots/youbot_gazebo.xacro" />
   <!-- Now we can start using the macros included above to define the actual youbot -->
-  <xacro:youbot_base name="base"/>
-  <xacro:joint_state_publisher />
+  <xacro:youbot_base name="base" namespace=""/>
+  <xacro:joint_state_publisher namespace=""/>
 </robot>

File: luh_youbot_description/robots/youbot_gazebo.xacro (robot description, xacro)
@@ -1,8 +1,8 @@
 <?xml version="1.0"?>
 <robot xmlns:xacro="http://ros.org/wiki/xacro">
-  <xacro:macro name="joint_state_publisher">
+  <xacro:macro name="joint_state_publisher" params="namespace">
   <gazebo>
       <plugin name="youbot_joint_state_publisher" filename="libyoubot_joint_state_publisher.so">
- 	<robotNamespace>gazebo</robotNamespace>
+ 	<robotNamespace>${namespace}</robotNamespace>
  	<updateRate>100.0</updateRate>
  	<alwaysOn>true</alwaysOn>

File: luh_youbot_description/urdf/youbot_arm/arm.urdf.xacro (robot description, xacro)
@@ -3,5 +3,5 @@
 	<xacro:include filename="$(find luh_youbot_description)/urdf/youbot_arm/limits.urdf.xacro" />
 	<xacro:include filename="$(find luh_youbot_description)/urdf/youbot_arm/arm.gazebo.xacro" />
-	<xacro:macro name="youbot_arm" params="parent name *origin">
+	<xacro:macro name="youbot_arm" params="parent name namespace *origin">
 		<!-- joint between base_link and arm_0_link -->
 		<joint name="${name}_joint_0" type="fixed" >
@@ -162,16 +162,15 @@
 				<origin xyz="0.003 0 -0.034" rpy="0 0 0" />
 				<geometry>
-					<mesh filename="package://luh_youbot_description/meshes/youbot_arm/arm5.dae" />
+					<mesh filename="package://luh_youbot_description/meshes/youbot_arm/arm5_new.dae" />
 				</geometry>
-				<material name="DarkGrey" />
 			</visual>
 			<collision>
 				<origin xyz="0.003 0 -0.034" rpy="0 0 0" />
 				<geometry>
-					<mesh filename="package://luh_youbot_description/meshes/youbot_arm/arm5_convex.dae" />
+					<mesh filename="package://luh_youbot_description/meshes/youbot_arm/arm5_new_convex.dae" />
 				</geometry>
 			</collision>
 		</link>
-                <xacro:youbot_arm_controller />
+                <xacro:youbot_arm_controller namespace="${namespace}"/>
 	</xacro:macro>
 </robot>

File: luh_youbot_description/urdf/youbot_base/base.gazebo.xacro (robot description, xacro)
@@ -1,8 +1,8 @@
 <?xml version="1.0"?>
 <robot xmlns:xacro="http://ros.org/wiki/xacro">
-  <xacro:macro name="youbot_base_controller">
+  <xacro:macro name="youbot_base_controller" params="namespace">
     <gazebo>
       <plugin name="base_controller" filename="libyoubot_base_controller.so">
-        <commandTopic>cmd_vel</commandTopic>
+        <commandTopic>${namespace}/cmd_vel</commandTopic>
         <odometryTopic>odom</odometryTopic>
         <odometryFrame>odom</odometryFrame>

File: luh_youbot_description/urdf/youbot_base/base.urdf.xacro (robot description, xacro)
@@ -20,5 +20,5 @@
 	<property name="wheel_joint_velocity" value="10" />
 	<property name="wheel_joint_safety_k_velocity" value="10.0" />
-	<xacro:macro name="youbot_base" params="name">
+	<xacro:macro name="youbot_base" params="name namespace">
 		<link name="${name}_footprint">
       			<visual>
@@ -190,5 +190,5 @@
       			</collision>
     		</link>
-                <xacro:youbot_base_controller/>
+                <xacro:youbot_base_controller namespace="${namespace}"/>
 	</xacro:macro>
 </robot>

File: luh_youbot_description/urdf/youbot_gripper/gripper.gazebo.xacro (robot description, xacro)
@@ -1,7 +1,7 @@
 <?xml version="1.0"?>
 <robot xmlns:xacro="http://ros.org/wiki/xacro">
-  <xacro:macro name="youbot_arm_controller" params="namespace">
+  <xacro:macro name="youbot_gripper_controller" params="namespace">
     <gazebo>
-      <plugin name="arm_controller" filename="libyoubot_arm_controller.so">
+      <plugin name="gripper_controller" filename="libyoubot_gripper_controller.so">
          <namespace>${namespace}</namespace>
       </plugin>

File: luh_youbot_description/urdf/youbot_gripper/gripper.urdf.xacro (robot description, xacro)
@@ -2,5 +2,6 @@
 <robot xmlns:xacro="http://ros.org/wiki/xacro">
 	<xacro:include filename="$(find luh_youbot_description)/urdf/youbot_gripper/limits.urdf.xacro" />
-	<xacro:macro name="youbot_gripper" params="parent name *origin">
+	<xacro:include filename="$(find luh_youbot_description)/urdf/youbot_gripper/gripper.gazebo.xacro" />
+	<xacro:macro name="youbot_gripper" params="parent name namespace *origin">
 		<!-- joint between arm_7_link and sdh_palm_link -->
 		<joint name="${name}_palm_joint" type="fixed" >
@@ -10,15 +11,15 @@
 		</joint>
 		<link name="${name}_palm_link">
-			<inertial>
+			<!--inertial>
 				<origin xyz="0 0 0" rpy="0 0 0"/>
 				<mass value="0.1"/>
 				<inertia ixx="0.01" ixy="0" ixz="0" iyy="0.01" iyz="0" izz="0.01" />
-			</inertial>
-			<visual>
+			</inertial-->
+			<!--visual>
 				<origin xyz="0 0 -0.0139" rpy="0 ${-M_PI/2} ${M_PI/2}"/>
 				<geometry>
 					<mesh filename="package://luh_youbot_description/meshes/youbot_gripper/palm.dae" />
 				</geometry>
-			</visual>
+			</visual-->
 			<!--collision>
 				<origin xyz="0.003 0 0.01" rpy="0 0 0" />
@@ -29,8 +30,8 @@
 		</link>
 		<joint name="${name}_finger_joint_l" type="prismatic">
-			<origin xyz="0.004 -0.002 0.046" rpy="0 0 0" />
+			<origin xyz="0.004 0.007 0.0115" rpy="0 0 ${M_PI}" />
 			<parent link="${name}_palm_link"/>
 			<child link="${name}_finger_link_l"/>
-			<axis xyz="0 1 0" />
+			<axis xyz="0 -1 0" />
 			<dynamics damping="1.0" friction="1.0" />
 			<limit effort="1" velocity="0.1" lower="0" upper="${finger_joint}"/>
@@ -44,5 +45,5 @@
 			</inertial>
 			<visual>
-				<origin xyz="0 -0.015 -0.02" rpy="0 ${-M_PI/2} 0" /> <!---->
+				<origin xyz="0 0 0" rpy="0 ${-M_PI/2} 0" /> <!---->
 				<geometry>
 					<mesh filename="package://luh_youbot_description/meshes/youbot_gripper/finger.dae" />
@@ -50,5 +51,5 @@
 			</visual>
 			<collision>
-				<origin xyz="0 -0.015 -0.02" rpy="0 ${-M_PI/2} 0" />
+				<origin xyz="0 0 0" rpy="0 ${-M_PI/2} 0" />
 				<geometry>
 					<mesh filename="package://luh_youbot_description/meshes/youbot_gripper/finger_convex.dae" />
@@ -57,8 +58,8 @@
 		</link>
                <joint name="${name}_finger_joint_r" type="prismatic">
-			<origin xyz="0.004 0.002 0.046" rpy="0 0 ${M_PI}" />
+			<origin xyz="0.004 -0.007 0.0115" rpy="0 0 0" />
 			<parent link="${name}_palm_link"/>
 			<child link="${name}_finger_link_r"/>
-			<axis xyz="0 1 0" />
+			<axis xyz="0 -1 0" />
 			<dynamics damping="1.0" friction="1.0" />
 			<limit effort="1" velocity="0.1" lower="0" upper="${finger_joint}"/>
@@ -72,5 +73,5 @@
 			</inertial>
 			<visual>
-				<origin xyz="0 -0.015 -0.02" rpy="0 ${-M_PI/2} 0" /> <!-- -->
+				<origin xyz="0 0 0" rpy="0 ${-M_PI/2} 0" /> <!-- -->
 				<geometry>
 					<mesh filename="package://luh_youbot_description/meshes/youbot_gripper/finger.dae" />
@@ -78,5 +79,5 @@
 			</visual>
 			<collision>
-				<origin xyz="0 -0.015 -0.02" rpy="0 ${-M_PI/2} 0" />
+				<origin xyz="0 0 0" rpy="0 ${-M_PI/2} 0" />
 				<geometry>
 					<mesh filename="package://luh_youbot_description/meshes/youbot_gripper/finger_convex.dae" />
@@ -97,4 +98,5 @@
 			</inertial>
 		</link>
+                <xacro:youbot_gripper_controller namespace="${namespace}"/>
 	</xacro:macro>
 </robot>

File: luh_youbot_description/urdf/youbot_gripper/limits.urdf.xacro (robot description, xacro)
@@ -5,5 +5,5 @@
         <property name="threshold" value="0.001" />
 	<!-- fingers limits, values are in meters -->
-	<property name="finger_joint" value="${0.023 / 2.0}" />
-	<property name="finger_joint_soft" value="${(0.023 - threshold) / 2.0}" />
+	<property name="finger_joint" value="${0.06 / 2.0}" />
+	<property name="finger_joint_soft" value="${(0.06 - threshold) / 2.0}" />
 </robot>

Commit message: added cam to gazebo

File: luh_youbot_description/robots/youbot.urdf.xacro (robot description, xacro)
@@ -15,9 +15,9 @@
   <xacro:include filename="$(find luh_youbot_description)/robots/youbot_gazebo.xacro" />
   <!-- Now we can start using the macros included above to define the actual youbot -->
-  <xacro:youbot_base name="base" namespace="gazebo"/>
+  <xacro:youbot_base name="base" namespace=""/>
   <xacro:youbot_plate name="plate" parent="base_link">
     <origin xyz="-0.039 0 0.064" rpy="0 0 0" />
   </xacro:youbot_plate>
-  <xacro:youbot_arm name="arm" parent="base_link" namespace="gazebo">
+  <xacro:youbot_arm name="arm" parent="base_link" namespace="">
     <origin xyz="0.258 0 0.066" rpy="0 0 0.576" />
   </xacro:youbot_arm>
@@ -25,4 +25,9 @@
     <origin xyz="0 0 0" rpy="0 0 0" />
   </xacro:youbot_gripper>
+  <!-- Kamera -->
+  <xacro:include filename="$(find luh_youbot_description)/urdf/sensors/asus_xtion_camera.urdf.xacro" />
+  <xacro:asus_xtion_camera name="cam3d" parent="arm_link_5" tilt="0.0">
+    <origin xyz="-0.02 0 -0.04" rpy="0 -1.60 0" />
+  </xacro:asus_xtion_camera>
   <xacro:joint_state_publisher namespace="gazebo"/>
 </robot>

File: luh_youbot_description/urdf/youbot_arm/arm.urdf.xacro (robot description, xacro)
@@ -159,5 +159,5 @@
 				<xacro:link_5_inertia_tensor />
 			</inertial>
-			<visual>
+				<visual>
 				<origin xyz="0.003 0 -0.034" rpy="0 0 0" />
 				<geometry>

Commit message: Quick fix for Arm jittering

File: luh_youbot_description/robots/youbot.urdf.xacro (robot description, xacro)
@@ -18,10 +18,16 @@
   <xacro:youbot_plate name="plate" parent="base_link">
     <origin xyz="-0.039 0 0.064" rpy="0 0 0" />
+    <!--Default inertia to see if jittering stops-->
+    <!--<inertia ixx="0.1" ixy="0" ixz="0" iyy="0.1" iyz="0" izz="0.1" />-->
   </xacro:youbot_plate>
   <xacro:youbot_arm name="arm" parent="base_link" namespace="">
     <origin xyz="0.258 0 0.066" rpy="0 0 0.576" />
+    <!--Default inertia to see if jittering stops-->
+    <!--<inertia ixx="0.1" ixy="0" ixz="0" iyy="0.1" iyz="0" izz="0.1" />-->
   </xacro:youbot_arm>
   <xacro:youbot_gripper name="gripper" parent="arm_link_5" namespace="">
     <origin xyz="0 0 0" rpy="0 0 0" />
+    <!--Default inertia to see if jittering stops-->
+    <!--<inertia ixx="0.1" ixy="0" ixz="0" iyy="0.1" iyz="0" izz="0.1" />-->
   </xacro:youbot_gripper>
   <!-- Kamera -->
@@ -29,4 +35,6 @@
   <xacro:asus_xtion_camera name="cam3d" parent="arm_link_5" tilt="0.0">
     <origin xyz="-0.02 0 -0.04" rpy="0 -1.60 0" />
+    <!--Default inertia to see if jittering stops-->
+    <!--<inertia ixx="0.1" ixy="0" ixz="0" iyy="0.1" iyz="0" izz="0.1" />-->
   </xacro:asus_xtion_camera>
   <xacro:joint_state_publisher namespace="gazebo"/>

File: luh_youbot_description/urdf/youbot_arm/arm.urdf.xacro (robot description, xacro)
@@ -9,9 +9,12 @@
 			<parent link="${parent}" />
 			<child link="${name}_link_0" />
+            <!--without Dynamics maybe causes jittering-->
+			<dynamics damping="1" friction="1" />
 		</joint>
 		<link name="${name}_link_0">
 			<inertial>
 				<origin xyz="0 0 0" rpy="0 0 0"/>
-				<mass value="${link_0_mass}"/>
+				<!--<mass value="${link_0_mass}"/>-->
+				<mass value="0.845"/>
 				<inertia ixx="0.01" ixy="0" ixz="0" iyy="0.01" iyz="0" izz="0.01" />
 			</inertial>
@@ -41,6 +44,10 @@
 		<link name="${name}_link_1">
 			<inertial>
-				<mass value="${link_1_mass}"/>
-				<xacro:link_1_inertia_tensor />
+                <!--See if this cause arm-jittering -->
+				<!--<mass value="${link_1_mass}"/>-->
+				<mass value="2.412"/>
+                <!-- looks like this is not loaded try with default-->
+				<!--<xacro:link_1_inertia_tensor />-->
+                <inertia ixx="0.003863" ixy="-0.000979" ixz="0.000000" iyy="0.006196" iyz="0.000000" izz="0.006369" />
 			</inertial>
 			<visual>
@@ -69,6 +76,9 @@
 		<link name="${name}_link_2">
 			<inertial>
-				<mass value="${link_2_mass}"/>
-				<xacro:link_2_inertia_tensor />
+                <!--See if this cause arm-jittering -->
+				<!--<mass value="${link_2_mass}"/>-->
+				<mass value="1.155"/>
+				<!--<xacro:link_2_inertia_tensor />-->
+                <inertia ixx="0.000823" ixy="0.000000" ixz="-0.000000" iyy="0.004447" iyz ="0.000000" izz="0.004439" />
 			</inertial>
 			<visual>
@@ -98,6 +108,9 @@
 		<link name="${name}_link_3">
 			<inertial>
-				<mass value="${link_3_mass}"/>
-				<xacro:link_3_inertia_tensor />
+                <!--See if this cause arm-jittering -->
+				<!--<mass value="${link_3_mass}"/>-->
+				<mass value="0.934"/>
+				<!--<xacro:link_3_inertia_tensor />-->
+				<inertia ixx="0.002459" ixy="0.000000" ixz="0.000000" iyy="0.002571" iyz="-0.000000" izz="0.000535" />
 			</inertial>
 			<visual>
@@ -127,6 +140,9 @@
 		<link name="${name}_link_4">
 			<inertial>
-				<mass value="${link_4_mass}"/>
-				<xacro:link_4_inertia_tensor />
+                <!--See if this cause arm-jittering -->
+				<!--<mass value="${link_4_mass}"/>-->
+				<mass value="0.877"/>
+				<!--<xacro:link_4_inertia_tensor />-->
+				<inertia ixx="0.000869" ixy="0.000000" ixz="-0.000000" iyy="0.001173" iyz="-0.000231" izz="0.001091" />
 			</inertial>
 			<visual>
@@ -156,6 +172,9 @@
 		<link name="${name}_link_5">
 			<inertial>
-				<mass value="${link_5_mass}"/>
-				<xacro:link_5_inertia_tensor />
+                <!--See if this cause arm-jittering -->
+				<!--<mass value="${link_5_mass}"/>-->
+				<mass value="0.251"/>
+				<!--<xacro:link_5_inertia_tensor />-->
+				<inertia ixx="0.000280" ixy="0.000000" ixz="0.000000" iyy="0.000339" iyz="0.000000" izz="0.000119" />
 			</inertial>
 				<visual>

File: luh_youbot_description/urdf/youbot_arm/limits.urdf.xacro (robot description, xacro)
@@ -25,4 +25,6 @@
 	<xacro:macro name="default_origin">
         	<origin xyz="0 0 0" rpy="0 0 0"/> <!-- no data known -->
+            <!--Default inertia to see -->
+            <inertia ixx="0.1" ixy="0" ixz="0" iyy="0.1" iyz="0" izz="0.1" />
 	</xacro:macro>
 	<xacro:macro name="link_default_inertia_tensor">

Commit message: Change Namespace of Gazebo-Camera_Topic due to testing barrier_detection, minor changes of inertia cause of jittering problems

File: luh_youbot_description/robots/youbot.urdf.xacro (robot description, xacro)
@@ -33,8 +33,8 @@
   <!-- Kamera -->
   <xacro:include filename="$(find luh_youbot_description)/urdf/sensors/asus_xtion_camera.urdf.xacro" />
-  <xacro:asus_xtion_camera name="cam3d" parent="arm_link_5" tilt="0.0">
+  <xacro:asus_xtion_camera name="camera" parent="arm_link_5" tilt="0.0">
     <origin xyz="-0.02 0 -0.04" rpy="0 -1.60 0" />
     <!--Default inertia to see if jittering stops-->
-    <!--<inertia ixx="0.1" ixy="0" ixz="0" iyy="0.1" iyz="0" izz="0.1" />-->
+    <inertia ixx="0.1" ixy="0" ixz="0" iyy="0.1" iyz="0" izz="0.1" />
   </xacro:asus_xtion_camera>
   <xacro:joint_state_publisher namespace="gazebo"/>

File: luh_youbot_description/urdf/youbot_gripper/gripper.urdf.xacro (robot description, xacro)
@@ -11,21 +11,21 @@
 		</joint>
 		<link name="${name}_palm_link">
-			<!--inertial>
+			<inertial>
 				<origin xyz="0 0 0" rpy="0 0 0"/>
 				<mass value="0.1"/>
 				<inertia ixx="0.01" ixy="0" ixz="0" iyy="0.01" iyz="0" izz="0.01" />
-			</inertial-->
-			<!--visual>
+			</inertial>
+			<visual>
 				<origin xyz="0 0 -0.0139" rpy="0 ${-M_PI/2} ${M_PI/2}"/>
 				<geometry>
 					<mesh filename="package://luh_youbot_description/meshes/youbot_gripper/palm.dae" />
 				</geometry>
-			</visual-->
-			<!--collision>
+			</visual>
+			<collision>
 				<origin xyz="0.003 0 0.01" rpy="0 0 0" />
 				<geometry>
 					<mesh filename="package://luh_youbot_description/meshes/youbot_gripper/palm_convex.dae" />
 				</geometry>
-			</collision-->
+			</collision>
 		</link>
 		<joint name="${name}_finger_joint_l" type="prismatic">

Commit message: tf bugfix

File: luh_youbot_description/robots/youbot.urdf.xacro (robot description, xacro)
@@ -18,6 +18,6 @@
   <xacro:youbot_plate name="plate" parent="base_link">
     <origin xyz="-0.039 0 0.064" rpy="0 0 0" />
-    <!--Default inertia to see if jittering stops-->
-    <!--<inertia ixx="0.1" ixy="0" ixz="0" iyy="0.1" iyz="0" izz="0.1" />-->
+    <!--Default inertia to see if  stops-->
+    <!--<inertia ixx="0.1" ixy="0" ijitteringxz="0" iyy="0.1" iyz="0" izz="0.1" />-->
   </xacro:youbot_plate>
   <xacro:youbot_arm name="arm" parent="base_link" namespace="">
@@ -31,11 +31,11 @@
     <!--<inertia ixx="0.1" ixy="0" ixz="0" iyy="0.1" iyz="0" izz="0.1" />-->
   </xacro:youbot_gripper>
-  <!-- Kamera -->
+  <!-- Kamera
   <xacro:include filename="$(find luh_youbot_description)/urdf/sensors/asus_xtion_camera.urdf.xacro" />
   <xacro:asus_xtion_camera name="camera" parent="arm_link_5" tilt="0.0">
     <origin xyz="-0.02 0 -0.04" rpy="0 -1.60 0" />
-    <!--Default inertia to see if jittering stops-->
     <inertia ixx="0.1" ixy="0" ixz="0" iyy="0.1" iyz="0" izz="0.1" />
   </xacro:asus_xtion_camera>
+-->
   <xacro:joint_state_publisher namespace="gazebo"/>
 </robot>
