Commit message: cleaned up and merged with latest master

File: luh_youbot_description/robots/youbot.urdf.xacro (robot description, xacro)
@@ -18,6 +18,6 @@
   <xacro:youbot_plate name="plate" parent="base_link">
     <origin xyz="-0.039 0 0.064" rpy="0 0 0" />
-    <!--Default inertia to see if jittering stops-->
-    <!--<inertia ixx="0.1" ixy="0" ixz="0" iyy="0.1" iyz="0" izz="0.1" />-->
+    <!--Default inertia to see if  stops-->
+    <!--<inertia ixx="0.1" ixy="0" ijitteringxz="0" iyy="0.1" iyz="0" izz="0.1" />-->
   </xacro:youbot_plate>
   <xacro:youbot_arm name="arm" parent="base_link" namespace="">
@@ -31,10 +31,10 @@
     <!--<inertia ixx="0.1" ixy="0" ixz="0" iyy="0.1" iyz="0" izz="0.1" />-->
   </xacro:youbot_gripper>
-  <!-- Kamera
-  <xacro:include filename="$(find luh_youbot_description)/urdf/sensors/asus_xtion_camera.urdf.xacro" />
+  <!-- Kamera -->
+  <!--xacro:include filename="$(find luh_youbot_description)/urdf/sensors/asus_xtion_camera.urdf.xacro" />
   <xacro:asus_xtion_camera name="camera" parent="arm_link_5" tilt="0.0">
     <origin xyz="-0.02 0 -0.04" rpy="0 -1.60 0" />
     <inertia ixx="0.1" ixy="0" ixz="0" iyy="0.1" iyz="0" izz="0.1" />
-  </xacro:asus_xtion_camera>-->
+  </xacro:asus_xtion_camera-->
   <xacro:joint_state_publisher namespace="gazebo"/>
 </robot>

File: luh_youbot_description/robots/youbot_gazebo.xacro (robot description, xacro)
@@ -1,8 +1,8 @@
 <?xml version="1.0"?>
-<robot xmlns:xacro="http://www.ros.org/wiki/xacro">
+<robot xmlns:xacro="http://ros.org/wiki/xacro">
   <xacro:macro name="joint_state_publisher" params="namespace">
     <gazebo>
         <plugin name="youbot_joint_state_publisher" filename="libyoubot_joint_state_publisher.so">
-         	<robotNamespace></robotNamespace>
+         	<robotNamespace>${namespace}</robotNamespace>
          	<updateRate>100.0</updateRate>
          	<alwaysOn>true</alwaysOn>

File: luh_youbot_description/urdf/common.xacro (robot description, xacro)
@@ -1,9 +1,9 @@
 <?xml version="1.0"?>
-<robot xmlns:xacro="http://www.ros.org/wiki/xacro">
-	<xacro:property name="M_PI" value="3.1415926535897931" />
+<robot>
+	<property name="M_PI" value="3.1415926535897931" />
 	<!-- Casters -->
-	<xacro:property name="cal_caster_fl" value="0.0" />
-	<xacro:property name="cal_caster_fr" value="0.0" />
-	<xacro:property name="cal_caster_bl" value="0.0" />
-	<xacro:property name="cal_caster_br" value="0.0" />
+	<property name="cal_caster_fl" value="0.0" />
+	<property name="cal_caster_fr" value="0.0" />
+	<property name="cal_caster_bl" value="0.0" />
+	<property name="cal_caster_br" value="0.0" />
 </robot>

File: luh_youbot_description/urdf/sensors/asus_xtion_camera.gazebo.xacro (robot description, xacro)
@@ -3,5 +3,5 @@
       xmlns:controller="http://playerstage.sourceforge.net/gazebo/xmlschema/#controller"
       xmlns:interface="http://playerstage.sourceforge.net/gazebo/xmlschema/#interface"
-      xmlns:xacro="http://www.ros.org/wiki/xacro">
+      xmlns:xacro="http://ros.org/wiki/xacro">
 <xacro:macro name="asus_xtion_camera_gazebo" params="name">
   <gazebo reference="${name}_camera">
@@ -17,6 +17,6 @@
       </image>
       <clip>
-        <near>0.1</near>
-        <far>5</far>
+        <near>0.05</near>
+        <far>3</far>
       </clip>
     </camera>
@@ -26,6 +26,9 @@
       <updateRate>20.0</updateRate>
       <cameraName>${name}_depth</cameraName>
-      <imageTopicName>/${name}/ir/image_raw</imageTopicName>
-      <cameraInfoTopicName>/${name}/ir/camera_info</cameraInfoTopicName>
+      <cameraName>${name}_rgb</cameraName>
+      <imageTopicName>/${name}/rgb/image_raw</imageTopicName>
+      <cameraInfoTopicName>/${name}/rgb/camera_info</cameraInfoTopicName>
+      <!--imageTopicName>/${name}/ir/image_raw</imageTopicName>
+      <cameraInfoTopicName>/${name}/ir/camera_info</cameraInfoTopicName-->
       <depthImageTopicName>/${name}/depth/image_raw</depthImageTopicName>
       <depthImageCameraInfoTopicName>/${name}/depth/camera_info</depthImageCameraInfoTopicName>
@@ -45,4 +48,5 @@
     </plugin>
   </sensor>
+<!--
   <sensor type="depth" name="${name}_rgb_frame_sensor">
     <always_on>true</always_on>
@@ -84,4 +88,5 @@
     </plugin>
   </sensor>
+-->
   </gazebo>
 </xacro:macro>

File: luh_youbot_description/urdf/sensors/asus_xtion_camera.urdf.xacro (robot description, xacro)
@@ -2,6 +2,6 @@
 <root xmlns:xacro="http://playerstage.sourceforge.net/gazebo/xmlschema/#interface">
   <xacro:include filename="$(find luh_youbot_description)/urdf/sensors/asus_xtion_camera.gazebo.xacro" />
-  <xacro:property name="eye_x_offset" value="0.03" />
-  <xacro:property name="eye_y_offset" value="0.035" />
+  <property name="eye_x_offset" value="0.03" />
+  <property name="eye_y_offset" value="0.035" />
   <xacro:macro name="asus_xtion_eye" params="suffix parent *origin">
 	<link name="${parent}_${suffix}_frame">
@@ -15,5 +15,5 @@
 	  <parent link="${parent}_camera"/>
 	  <child link="${parent}_${suffix}_frame"/>
-	  <xacro:insert_block name="origin"/>
+	  <insert_block name="origin"/>
 	</joint>
   </xacro:macro>
@@ -40,5 +40,5 @@
     </link>
     <joint name="${name}_foot_joint" type="fixed">
-      <xacro:insert_block name="origin" />
+      <insert_block name="origin" />
       <parent link="${parent}"/>
       <child link="${name}_foot_link"/>

File: luh_youbot_description/urdf/sensors/hokuyo_urg04_laser.gazebo.xacro (robot description, xacro)
@@ -1,4 +1,4 @@
 <?xml version="1.0"?>
-<robot xmlns:xacro="http://www.ros.org/wiki/xacro">
+<robot xmlns:xacro="http://ros.org/wiki/xacro">
   <xacro:macro name="hokuyo_urg04_laser_gazebo" params="name ros_topic update_rate min_angle max_angle">
     <gazebo reference="${name}_link">

File: luh_youbot_description/urdf/sensors/hokuyo_urg04_laser.urdf.xacro (robot description, xacro)
@@ -1,9 +1,9 @@
 <?xml version="1.0"?>
-<robot xmlns:xacro="http://www.ros.org/wiki/xacro">
+<robot xmlns:xacro="http://ros.org/wiki/xacro">
   <xacro:include filename="$(find luh_youbot_description)/urdf/sensors/hokuyo_urg04_laser.gazebo.xacro" />
   <xacro:macro name="hokuyo_urg04_laser" params="name parent *origin ros_topic update_rate min_angle max_angle">
     <joint name="${name}_hokuyo_urg04_laser_joint" type="fixed">
       <axis xyz="0 1 0" />
-      <xacro:insert_block name="origin" />
+      <insert_block name="origin" />
       <parent link="${parent}_link"/>
       <child link="${name}_link"/>

File: luh_youbot_description/urdf/sensors/kinect_camera.gazebo.xacro (robot description, xacro)
@@ -3,5 +3,5 @@
       xmlns:controller="http://playerstage.sourceforge.net/gazebo/xmlschema/#controller"
       xmlns:interface="http://playerstage.sourceforge.net/gazebo/xmlschema/#interface"
-      xmlns:xacro="http://www.ros.org/wiki/xacro">
+      xmlns:xacro="http://ros.org/wiki/xacro">
 <xacro:macro name="kinect_camera_gazebo" params="name">
   <gazebo reference="${name}_camera">

File: luh_youbot_description/urdf/sensors/kinect_camera.urdf.xacro (robot description, xacro)
@@ -3,9 +3,9 @@
       xmlns:controller="http://playerstage.sourceforge.net/gazebo/xmlschema/#controller"
       xmlns:interface="http://playerstage.sourceforge.net/gazebo/xmlschema/#interface"
-      xmlns:xacro="http://www.ros.org/wiki/xacro">
+      xmlns:xacro="http://ros.org/wiki/xacro">
   <xacro:include filename="$(find luh_youbot_description)/urdf/sensors/kinect_camera.gazebo.xacro"/>
   <xacro:macro name="kinect_camera" params="name parent *origin">
    <joint name="${name}_camera_joint" type="fixed">
-    <xacro:insert_block name="origin" />
+    <insert_block name="origin" />
     <parent link="${parent}" />
     <child link="${name}_camera" />

File: luh_youbot_description/urdf/sensors/microsoft_lifecam.gazebo.xacro (robot description, xacro)
@@ -3,5 +3,5 @@
       xmlns:controller="http://playerstage.sourceforge.net/gazebo/xmlschema/#controller"
       xmlns:interface="http://playerstage.sourceforge.net/gazebo/xmlschema/#interface"
-      xmlns:xacro="http://www.ros.org/wiki/xacro">
+      xmlns:xacro="http://ros.org/wiki/xacro">
 <xacro:macro name="microsoft_lifecam_gazebo" params="name">
   <gazebo reference="${name}_camera">

File: luh_youbot_description/urdf/sensors/microsoft_lifecam.urdf.xacro (robot description, xacro)
@@ -3,9 +3,9 @@
       xmlns:controller="http://playerstage.sourceforge.net/gazebo/xmlschema/#controller"
       xmlns:interface="http://playerstage.sourceforge.net/gazebo/xmlschema/#interface"
-      xmlns:xacro="http://www.ros.org/wiki/xacro">
+      xmlns:xacro="http://ros.org/wiki/xacro">
   <xacro:include filename="$(find luh_youbot_description)/urdf/sensors/microsoft_lifecam.gazebo.xacro"/>
   <xacro:macro name="microsoft_lifecam" params="name parent *origin">
    <joint name="${name}_camera_joint" type="fixed">
-    <xacro:insert_block name="origin" />
+    <insert_block name="origin" />
     <parent link="${parent}" />
     <child link="${name}_camera" />

File: luh_youbot_description/urdf/youbot_arm/arm.gazebo.xacro (robot description, xacro)
@@ -1,8 +1,8 @@
 <?xml version="1.0"?>
-<robot xmlns:xacro="http://www.ros.org/wiki/xacro">
+<robot xmlns:xacro="http://ros.org/wiki/xacro">
   <xacro:macro name="youbot_arm_controller" params="namespace">
     <gazebo>
       <plugin name="arm_controller" filename="libyoubot_arm_controller.so">
-         <namespace></namespace>
+         <namespace>${namespace}</namespace>
       </plugin>
    </gazebo>

File: luh_youbot_description/urdf/youbot_arm/arm.urdf.xacro (robot description, xacro)
@@ -1,4 +1,4 @@
 <?xml version="1.0"?>
-<robot  xmlns:xacro="http://www.ros.org/wiki/xacro">
+<robot  xmlns:xacro="http://ros.org/wiki/xacro">
 	<xacro:include filename="$(find luh_youbot_description)/urdf/youbot_arm/limits.urdf.xacro" />
 	<xacro:include filename="$(find luh_youbot_description)/urdf/youbot_arm/arm.gazebo.xacro" />
@@ -6,5 +6,5 @@
 		<!-- joint between base_link and arm_0_link -->
 		<joint name="${name}_joint_0" type="fixed" >
-			<xacro:insert_block name="origin" />
+			<insert_block name="origin" />
 			<parent link="${parent}" />
 			<child link="${name}_link_0" />
@@ -12,4 +12,10 @@
 			<dynamics damping="1" friction="1" />
 		</joint>
+                <joint name="${name}_joint_origin" type="fixed" >
+                        <origin xyz="0.024 0 0.0" rpy="0 0 0"/>
+			<parent link="${name}_link_0" />
+			<child link="${name}_origin" />
+		</joint>
+		<link name="${name}_origin"/>
 		<link name="${name}_link_0">
 			<inertial>
@@ -191,5 +197,5 @@
 			</collision>
 		</link>
-                <xacro:youbot_arm_controller namespace="${namespace}"/>
+                <xacro:youbot_arm_controller namespace="gazebo"/>
 	</xacro:macro>
 </robot>

File: luh_youbot_description/urdf/youbot_arm/limits.urdf.xacro (robot description, xacro)
@@ -1,25 +1,25 @@
 <?xml version="1.0"?>
-<robot xmlns:xacro="http://www.ros.org/wiki/xacro">>
+<robot xmlns:xacro="http://ros.org/wiki/xacro">>
 	<!-- common properties -->
-	<xacro:property name="M_PI" value="3.1415926535897931" />
-        <xacro:property name="threshold" value="0.01" />
+	<property name="M_PI" value="3.1415926535897931" />
+        <property name="threshold" value="0.01" />
 	<!-- arm limits positions (deg) -->
-	<xacro:property name="joint_1_limit" value="${M_PI * (169 + 169) / 180}" />
-	<xacro:property name="joint_2_limit" value="${M_PI * (90 + 65) / 180}" />
-	<xacro:property name="joint_3_limit" value="${M_PI * (146 + 151) / 180}" />
-	<xacro:property name="joint_4_limit" value="${M_PI * (102.5 + 102.5) / 180}" />
-	<xacro:property name="joint_5_limit" value="${M_PI * (167.5 + 167.5) / 180}" />
-        <xacro:property name="joint_1_limit_soft" value="${M_PI * (169 + 169) / 180 - threshold}" />
-	<xacro:property name="joint_2_limit_soft" value="${M_PI * (90 + 65) / 180 - threshold}" />
-	<xacro:property name="joint_3_limit_soft" value="${M_PI * (146 + 151) / 180 - threshold}" />
-	<xacro:property name="joint_4_limit_soft" value="${M_PI * (102.5 + 102.5) / 180 - threshold}" />
-	<xacro:property name="joint_5_limit_soft" value="${M_PI * (167.5 + 167.5) / 180 - threshold}" />
+	<property name="joint_1_limit" value="${M_PI * (169 + 169) / 180}" />
+	<property name="joint_2_limit" value="${M_PI * (90 + 65) / 180}" />
+	<property name="joint_3_limit" value="${M_PI * (146 + 151) / 180}" />
+	<property name="joint_4_limit" value="${M_PI * (102.5 + 102.5) / 180}" />
+	<property name="joint_5_limit" value="${M_PI * (167.5 + 167.5) / 180}" />
+        <property name="joint_1_limit_soft" value="${M_PI * (169 + 169) / 180 - threshold}" />
+	<property name="joint_2_limit_soft" value="${M_PI * (90 + 65) / 180 - threshold}" />
+	<property name="joint_3_limit_soft" value="${M_PI * (146 + 151) / 180 - threshold}" />
+	<property name="joint_4_limit_soft" value="${M_PI * (102.5 + 102.5) / 180 - threshold}" />
+	<property name="joint_5_limit_soft" value="${M_PI * (167.5 + 167.5) / 180 - threshold}" />
 	<!-- dynamic properties : mass (kg) Alu data sheet -->
-	<xacro:property name="link_0_mass" value="0.845" />
-	<xacro:property name="link_1_mass" value="2.412" />
-	<xacro:property name="link_2_mass" value="1.155" />
-	<xacro:property name="link_3_mass" value="0.934" />
-	<xacro:property name="link_4_mass" value="0.877" />
-	<xacro:property name="link_5_mass" value="0.251" />
+	<property name="link_0_mass" value="0.845" />
+	<property name="link_1_mass" value="2.412" />
+	<property name="link_2_mass" value="1.155" />
+	<property name="link_3_mass" value="0.934" />
+	<property name="link_4_mass" value="0.877" />
+	<property name="link_5_mass" value="0.251" />
 	<!-- TODO: add inertia tensor-->
 	<xacro:macro name="default_origin">

File: luh_youbot_description/urdf/youbot_base/base.gazebo.xacro (robot description, xacro)
@@ -1,8 +1,8 @@
 <?xml version="1.0"?>
-<robot xmlns:xacro="http://www.ros.org/wiki/xacro">
+<robot xmlns:xacro="http://ros.org/wiki/xacro">
   <xacro:macro name="youbot_base_controller" params="namespace">
     <gazebo>
       <plugin name="base_controller" filename="libyoubot_base_controller.so">
-        <commandTopic>/cmd_vel</commandTopic>
+        <commandTopic>${namespace}/cmd_vel</commandTopic>
         <odometryTopic>odom</odometryTopic>
         <odometryFrame>odom</odometryFrame>

File: luh_youbot_description/urdf/youbot_base/base.urdf.xacro (robot description, xacro)
@@ -1,24 +1,24 @@
 <?xml version="1.0"?>
-<robot  xmlns:xacro="http://www.ros.org/wiki/xacro">
+<robot  xmlns:xacro="http://ros.org/wiki/xacro">
 	<!-- sensors -->
 	<xacro:include filename="$(find luh_youbot_description)/urdf/sensors/hokuyo_urg04_laser.urdf.xacro"/>
-  	<xacro:include filename="$(find luh_youbot_description)/urdf/youbot_base/base.gazebo.xacro" />
-  	<xacro:include filename="$(find luh_youbot_description)/urdf/youbot_base/bumper.gazebo.xacro" />
+  <xacro:include filename="$(find luh_youbot_description)/urdf/youbot_base/base.gazebo.xacro" />
+  <xacro:include filename="$(find luh_youbot_description)/urdf/youbot_base/bumper.gazebo.xacro" />
  	<!-- simplified box collision geometry for base -->
-  	<xacro:property name="base_size_x" value="0.570" />
-  	<xacro:property name="base_size_y" value="0.40" />
-  	<xacro:property name="base_size_z" value="0.100" />
-	<xacro:property name="base_mass" value="22.0" />
-	<xacro:property name="wheel_offset_x" value="0.228"  />
-  	<xacro:property name="wheel_offset_y" value="0.158"  />
-  	<xacro:property name="wheel_offset_z" value="-0.034" />
-	<xacro:property name="wheel_mass" value="0.4" />
-	<xacro:property name="wheel_radius" value="0.05" />
-	<xacro:property name="wheel_length" value="0.07" />
-	<xacro:property name="wheel_joint_damping" value="0.0" />
-	<xacro:property name="wheel_joint_friction" value="0.0" />
-	<xacro:property name="wheel_joint_effort" value="30" />
-	<xacro:property name="wheel_joint_velocity" value="10" />
-	<xacro:property name="wheel_joint_safety_k_velocity" value="10.0" />
+  	<property name="base_size_x" value="0.570" />
+  	<property name="base_size_y" value="0.40" />
+  	<property name="base_size_z" value="0.100" />
+	  <property name="base_mass" value="22.0" />
+	<property name="wheel_offset_x" value="0.228"  />
+  	<property name="wheel_offset_y" value="0.158"  />
+  	<property name="wheel_offset_z" value="-0.034" />
+	<property name="wheel_mass" value="0.4" />
+	<property name="wheel_radius" value="0.05" />
+	<property name="wheel_length" value="0.07" />
+	<property name="wheel_joint_damping" value="0.0" />
+	<property name="wheel_joint_friction" value="0.0" />
+	<property name="wheel_joint_effort" value="30" />
+	<property name="wheel_joint_velocity" value="10" />
+	<property name="wheel_joint_safety_k_velocity" value="10.0" />
 	<xacro:macro name="youbot_base" params="name namespace">
 		<link name="${name}_footprint">
@@ -31,6 +31,5 @@
       			</visual>
       			<collision>
-				<!--<origin xyz="0 0 ${-base_size_z / 2.0}" rpy="0 0 0" />-->
-				<origin xyz="0 0 0.1" rpy="0 0 0" />
+        			<origin xyz="0 0 ${-base_size_z / 2.0}" rpy="0 0 0" />
         			<geometry>
           				<box size="0.001 0.001 0.001" />
@@ -39,5 +38,5 @@
     		</link>
     		<joint name="${name}_footprint_joint" type="fixed">
-      			<origin xyz="0 0 0.083" rpy="0 0 0" />
+      			<origin xyz="0 0 0" rpy="0 0 0" />
       			<child link="${name}_link" />
       			<parent link="${name}_footprint"/>
@@ -192,5 +191,5 @@
       			</collision>
     		</link>
-        <xacro:youbot_base_controller namespace="${namespace}"/>
+        <xacro:youbot_base_controller namespace="gazebo"/>
         <xacro:youbot_base_bumper namespace="${namespace}"/>
 	</xacro:macro>

File: luh_youbot_description/urdf/youbot_base/bumper.gazebo.xacro (robot description, xacro)
@@ -1,4 +1,4 @@
 <?xml version="1.0"?>
-<robot xmlns:xacro="http://www.ros.org/wiki/xacro">
+<robot xmlns:xacro="http://ros.org/wiki/xacro">
   <xacro:macro name="youbot_base_bumper" params="namespace">
   <gazebo reference="${name}_link">   <!--  -->

File: luh_youbot_description/urdf/youbot_gripper/gripper.gazebo.xacro (robot description, xacro)
@@ -1,4 +1,4 @@
 <?xml version="1.0"?>
-<robot xmlns:xacro="http://www.ros.org/wiki/xacro">
+<robot xmlns:xacro="http://ros.org/wiki/xacro">
   <xacro:macro name="youbot_gripper_controller" params="namespace">
     <gazebo>

File: luh_youbot_description/urdf/youbot_gripper/gripper.urdf.xacro (robot description, xacro)
@@ -1,4 +1,4 @@
 <?xml version="1.0"?>
-<robot xmlns:xacro="http://www.ros.org/wiki/xacro">
+<robot xmlns:xacro="http://ros.org/wiki/xacro">
 	<xacro:include filename="$(find luh_youbot_description)/urdf/youbot_gripper/limits.urdf.xacro" />
 	<xacro:include filename="$(find luh_youbot_description)/urdf/youbot_gripper/gripper.gazebo.xacro" />
@@ -6,5 +6,5 @@
 		<!-- joint between arm_7_link and sdh_palm_link -->
 		<joint name="${name}_palm_joint" type="fixed" >
-			<xacro:insert_block name="origin" />
+			<insert_block name="origin" />
 			<parent link="${parent}" />
 			<child link="${name}_palm_link" />
@@ -87,5 +87,5 @@
 		<!-- coordinate frame on the tip of the robot's gripper -->
 		<joint name="${name}_tip_joint" type="fixed">
-			<origin xyz="0.004 0 0.1" rpy="0.0 ${-M_PI / 2} 0.0" />
+			<origin xyz="0.000 0 0.09" rpy="0.0 ${-M_PI / 2} 0.0" />
 			<parent link="${name}_palm_link" />
 			<child link="${name}_tip"/>

File: luh_youbot_description/urdf/youbot_gripper/limits.urdf.xacro (robot description, xacro)
@@ -1,9 +1,9 @@
 <?xml version="1.0"?>
-<robot xmlns:xacro="http://www.ros.org/wiki/xacro">
+<robot>
 	<!-- common properties -->
-	<xacro:property name="M_PI" value="3.1415926535897931" />
-        <xacro:property name="threshold" value="0.001" />
+	<property name="M_PI" value="3.1415926535897931" />
+        <property name="threshold" value="0.001" />
 	<!-- fingers limits, values are in meters -->
-	<xacro:property name="finger_joint" value="${0.06 / 2.0}" />
-	<xacro:property name="finger_joint_soft" value="${(0.06 - threshold) / 2.0}" />
+	<property name="finger_joint" value="${0.06 / 2.0}" />
+	<property name="finger_joint_soft" value="${(0.06 - threshold) / 2.0}" />
 </robot>
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