Commit message: adjusted kinematic parameters 1. to match current gripper 2. to have same values in urdf as in kinematics lib

File: luh_youbot_description/urdf/youbot_arm/arm.urdf.xacro (robot description, xacro)
@@ -34,5 +34,5 @@
 		<!-- joint between arm_0_link and arm_1_link -->
 		<joint name="${name}_joint_1" type="revolute">
-			<origin xyz="0.024 0 0.096" rpy="0 0 ${170 * M_PI / 180}"/>
+			<origin xyz="0.024 0 0.096" rpy="0 0 2.949606436"/>
 			<parent link="${name}_link_0"/>
 			<child link="${name}_link_1"/>
@@ -66,5 +66,5 @@
 		<!-- joint between arm_1_link and arm_2_link -->
 		<joint name="${name}_joint_2" type="revolute">
-			<origin xyz="0.033 0 0.019" rpy="0 ${-65 * M_PI / 180} 0"/>
+			<origin xyz="0.033 0 0.019" rpy="0 -1.13446737019872 0"/>
 			<parent link="${name}_link_1"/>
 			<child link="${name}_link_2"/>
@@ -98,5 +98,5 @@
 		<!-- joint between arm_2_link and arm_3_link -->
 		<joint name="${name}_joint_3" type="revolute">
-			<origin xyz="0.000 0.000 0.155" rpy="0 ${146 * M_PI / 180} 0"/>
+			<origin xyz="0.000 0.000 0.155" rpy="0 2.54817721725322 0"/>
 			<parent link="${name}_link_2"/>
 			<child link="${name}_link_3"/>
@@ -130,5 +130,5 @@
 		<!-- joint between arm_3_link and arm_4_link -->
 		<joint name="${name}_joint_4" type="revolute">
-			<origin xyz="0.000 0.000 0.135" rpy="0 ${-102.5 * M_PI / 180} 0" />
+			<origin xyz="0.000 0.000 0.135" rpy="0 -1.78896002508397 0" />
 			<parent link="${name}_link_3"/>
 			<child link="${name}_link_4"/>
@@ -162,5 +162,5 @@
 		<!-- joint between arm_4_link and arm_5_link -->
 		<joint name="${name}_joint_5" type="revolute">
-			<origin xyz="-0.002 0 0.130" rpy="0 0 ${167.5 * M_PI / 180}" />
+			<origin xyz="0 0 0.130" rpy="0 0 3.00194664774853" />
 			<parent link="${name}_link_4"/>
 			<child link="${name}_link_5"/>

File: luh_youbot_description/urdf/youbot_gripper/gripper.urdf.xacro (robot description, xacro)
@@ -87,5 +87,5 @@
 		<!-- coordinate frame on the tip of the robot's gripper -->
 		<joint name="${name}_tip_joint" type="fixed">
-			<origin xyz="0.004 0 0.1" rpy="0.0 ${-M_PI / 2} 0.0" />
+			<origin xyz="0.000 0 0.09" rpy="0.0 ${-M_PI / 2} 0.0" />
 			<parent link="${name}_palm_link" />
 			<child link="${name}_tip"/>

Commit message: Changed arm.urdf.xacro, added arm_link_origin

File: luh_youbot_description/urdf/youbot_arm/arm.urdf.xacro (robot description, xacro)
@@ -12,4 +12,10 @@
 			<dynamics damping="1" friction="1" />
 		</joint>
+                <joint name="${name}_joint_origin" type="fixed" >
+                        <origin xyz="0.024 0 0.0" rpy="0 0 0"/>
+			<parent link="${name}_link_0" />
+			<child link="${name}_origin" />
+		</joint>
+		<link name="${name}_origin"/>
 		<link name="${name}_link_0">
 			<inertial>

Commit message: luh_youbot_description: added arm_origin

File: luh_youbot_description/urdf/youbot_arm/arm.urdf.xacro (robot description, xacro)
@@ -12,4 +12,10 @@
 			<dynamics damping="1" friction="1" />
 		</joint>
+                <joint name="${name}_joint_origin" type="fixed" >
+                        <origin xyz="0.024 0 0.0" rpy="0 0 0"/>
+			<parent link="${name}_link_0" />
+			<child link="${name}_origin" />
+		</joint>
+		<link name="${name}_origin"/>
 		<link name="${name}_link_0">
 			<inertial>
@@ -34,5 +40,5 @@
 		<!-- joint between arm_0_link and arm_1_link -->
 		<joint name="${name}_joint_1" type="revolute">
-			<origin xyz="0.024 0 0.096" rpy="0 0 2.949606436"/>
+			<origin xyz="0.024 0 0.096" rpy="0 0 ${170 * M_PI / 180}"/>
 			<parent link="${name}_link_0"/>
 			<child link="${name}_link_1"/>
@@ -66,5 +72,5 @@
 		<!-- joint between arm_1_link and arm_2_link -->
 		<joint name="${name}_joint_2" type="revolute">
-			<origin xyz="0.033 0 0.019" rpy="0 -1.13446737019872 0"/>
+			<origin xyz="0.033 0 0.019" rpy="0 ${-65 * M_PI / 180} 0"/>
 			<parent link="${name}_link_1"/>
 			<child link="${name}_link_2"/>
@@ -98,5 +104,5 @@
 		<!-- joint between arm_2_link and arm_3_link -->
 		<joint name="${name}_joint_3" type="revolute">
-			<origin xyz="0.000 0.000 0.155" rpy="0 2.54817721725322 0"/>
+			<origin xyz="0.000 0.000 0.155" rpy="0 ${146 * M_PI / 180} 0"/>
 			<parent link="${name}_link_2"/>
 			<child link="${name}_link_3"/>
@@ -130,5 +136,5 @@
 		<!-- joint between arm_3_link and arm_4_link -->
 		<joint name="${name}_joint_4" type="revolute">
-			<origin xyz="0.000 0.000 0.135" rpy="0 -1.78896002508397 0" />
+			<origin xyz="0.000 0.000 0.135" rpy="0 ${-102.5 * M_PI / 180} 0" />
 			<parent link="${name}_link_3"/>
 			<child link="${name}_link_4"/>
@@ -162,5 +168,5 @@
 		<!-- joint between arm_4_link and arm_5_link -->
 		<joint name="${name}_joint_5" type="revolute">
-			<origin xyz="0 0 0.130" rpy="0 0 3.00194664774853" />
+			<origin xyz="-0.002 0 0.130" rpy="0 0 ${167.5 * M_PI / 180}" />
 			<parent link="${name}_link_4"/>
 			<child link="${name}_link_5"/>
