Commit message: Collision Model youbot_base angepasst für Bumber-Collission-Detector

File: luh_youbot_description/urdf/youbot_base/base.urdf.xacro (robot description, xacro)
@@ -6,5 +6,5 @@
   <xacro:include filename="$(find luh_youbot_description)/urdf/youbot_base/bumper.gazebo.xacro" />
  	<!-- simplified box collision geometry for base -->
-  	<property name="base_size_x" value="0.750" />
+  	<property name="base_size_x" value="0.570" />
   	<property name="base_size_y" value="0.40" />
   	<property name="base_size_z" value="0.100" />
@@ -59,6 +59,5 @@
         			<origin xyz="0 0 0" rpy="0 0 0" />
         			<geometry>
-          				<box size="${base_size_x} ${base_size_y} ${base_size_z}" />
-			<!--		<mesh filename="package://luh_youbot_description/meshes/youbot_base/base_convex.dae"/>   -->
+					<mesh filename="package://luh_youbot_description/meshes/youbot_base/base_convex.dae"/>
 	       			</geometry>
       			</collision>

Commit message: URDF von base_ffot_print zu base_link angepasst

File: luh_youbot_description/urdf/youbot_base/base.urdf.xacro (robot description, xacro)
@@ -38,5 +38,5 @@
     		</link>
     		<joint name="${name}_footprint_joint" type="fixed">
-      			<origin xyz="0 0 0" rpy="0 0 0" />
+      			<origin xyz="0 0 0.083" rpy="0 0 0" />
       			<child link="${name}_link" />
       			<parent link="${name}_footprint"/>

Commit message: luh_youbot_description: fixed base.urdf

File: luh_youbot_description/urdf/youbot_base/base.urdf.xacro (robot description, xacro)
@@ -38,5 +38,5 @@
     		</link>
     		<joint name="${name}_footprint_joint" type="fixed">
-      			<origin xyz="0 0 0.083" rpy="0 0 0" />
+      			<origin xyz="0 0 0" rpy="0 0 0" />
       			<child link="${name}_link" />
       			<parent link="${name}_footprint"/>

Commit message: minor changes

File: luh_youbot_description/urdf/youbot_base/base.urdf.xacro (robot description, xacro)
@@ -31,5 +31,6 @@
       			</visual>
       			<collision>
-        			<origin xyz="0 0 ${-base_size_z / 2.0}" rpy="0 0 0" />
+				<!--<origin xyz="0 0 ${-base_size_z / 2.0}" rpy="0 0 0" />-->
+				<origin xyz="0 0 0.1" rpy="0 0 0" />
         			<geometry>
           				<box size="0.001 0.001 0.001" />
